Commit message: Added h1 skins for torso

File: robots/h1-2/skin/elbow_L_skin.xacro (robot description, xacro)
@@ -5,5 +5,5 @@
     <!-- Properties -->
     <xacro:property name="use_mesh_file" value="true" />
-    <xacro:property name="mesh_file" value="REPLACE_ME" />
+    <xacro:property name="mesh_file" value="package://gentact_descriptions/h1-2/meshes/skin/elbow_L_skin.stl" />
     <xacro:property name="mass" value="0.0" /> <!-- [kg] -->
     <xacro:property name="body_width" value="0.0" /> <!-- [m] -->

File: robots/h1-2/skin/elbow_R_skin.xacro (robot description, xacro)
@@ -5,5 +5,5 @@
     <!-- Properties -->
     <xacro:property name="use_mesh_file" value="true" />
-    <xacro:property name="mesh_file" value="REPLACE_ME" />
+    <xacro:property name="mesh_file" value="package://gentact_descriptions/h1-2/meshes/skin/elbow_R_skin.stl" />
     <xacro:property name="mass" value="0.0" /> <!-- [kg] -->
     <xacro:property name="body_width" value="0.0" /> <!-- [m] -->

File: robots/h1-2/skin/head_skin.xacro (robot description, xacro)
@@ -5,5 +5,5 @@
     <!-- Properties -->
     <xacro:property name="use_mesh_file" value="true" />
-    <xacro:property name="mesh_file" value="REPLACE_ME" />
+    <xacro:property name="mesh_file" value="package://gentact_descriptions/h1-2/meshes/skin/head_skin.stl" />
     <xacro:property name="mass" value="0.0" /> <!-- [kg] -->
     <xacro:property name="body_width" value="0.0" /> <!-- [m] -->

File: robots/h1-2/skin/shoulder_roll_L_skin.xacro (robot description, xacro)
@@ -5,5 +5,5 @@
     <!-- Properties -->
     <xacro:property name="use_mesh_file" value="true" />
-    <xacro:property name="mesh_file" value="REPLACE_ME" />
+    <xacro:property name="mesh_file" value="package://gentact_descriptions/h1-2/meshes/skin/shoulder_roll_L_skin.stl" />
     <xacro:property name="mass" value="0.0" /> <!-- [kg] -->
     <xacro:property name="body_width" value="0.0" /> <!-- [m] -->

File: robots/h1-2/skin/shoulder_roll_R_skin.xacro (robot description, xacro)
@@ -5,5 +5,5 @@
     <!-- Properties -->
     <xacro:property name="use_mesh_file" value="true" />
-    <xacro:property name="mesh_file" value="REPLACE_ME" />
+    <xacro:property name="mesh_file" value="package://gentact_descriptions/h1-2/meshes/skin/shoulder_roll_R_skin.stl" />
     <xacro:property name="mass" value="0.0" /> <!-- [kg] -->
     <xacro:property name="body_width" value="0.0" /> <!-- [m] -->

File: robots/h1-2/skin/shoulder_yaw_L_skin.xacro (robot description, xacro)
@@ -5,5 +5,5 @@
     <!-- Properties -->
     <xacro:property name="use_mesh_file" value="true" />
-    <xacro:property name="mesh_file" value="REPLACE_ME" />
+    <xacro:property name="mesh_file" value="package://gentact_descriptions/h1-2/meshes/skin/shoulder_yaw_L_skin.stl" />
     <xacro:property name="mass" value="0.0" /> <!-- [kg] -->
     <xacro:property name="body_width" value="0.0" /> <!-- [m] -->

File: robots/h1-2/skin/shoulder_yaw_R_skin.xacro (robot description, xacro)
@@ -5,5 +5,5 @@
     <!-- Properties -->
     <xacro:property name="use_mesh_file" value="true" />
-    <xacro:property name="mesh_file" value="REPLACE_ME" />
+    <xacro:property name="mesh_file" value="package://gentact_descriptions/h1-2/meshes/skin/shoulder_yaw_R_skin.stl" />
     <xacro:property name="mass" value="0.0" /> <!-- [kg] -->
     <xacro:property name="body_width" value="0.0" /> <!-- [m] -->

File: robots/h1-2/skin/torso_skin.xacro (robot description, xacro)
@@ -5,5 +5,5 @@
     <!-- Properties -->
     <xacro:property name="use_mesh_file" value="true" />
-    <xacro:property name="mesh_file" value="REPLACE_ME" />
+    <xacro:property name="mesh_file" value="package://gentact_descriptions/h1-2/meshes/skin/torso_skin.stl" />
     <xacro:property name="mass" value="0.0" /> <!-- [kg] -->
     <xacro:property name="body_width" value="0.0" /> <!-- [m] -->

Commit message: added h1

File: robots/h1-2/skin/elbow_L_skin.xacro (robot description, xacro)
@@ -2,8 +2,8 @@
 <robot xmlns:xacro="http://ros.org/wiki/xacro">
 <!-- Macro definition for skin unit -->
-<xacro:macro name="elbow_L_skin" params="parent namespace">
+<xacro:macro name="elbow_R_skin" params="parent namespace">
     <!-- Properties -->
     <xacro:property name="use_mesh_file" value="true" />
-    <xacro:property name="mesh_file" value="meshes/skin/elbow_L_skin.stl" />
+    <xacro:property name="mesh_file" value="meshes/skin/elbow_R_skin.stl" />
     <xacro:property name="mass" value="0.0" /> <!-- [kg] -->
     <xacro:property name="body_width" value="0.0" /> <!-- [m] -->

File: robots/h1-2/skin/elbow_R_skin.xacro (robot description, xacro)
@@ -2,8 +2,8 @@
 <robot xmlns:xacro="http://ros.org/wiki/xacro">
 <!-- Macro definition for skin unit -->
-<xacro:macro name="elbow_R_skin" params="parent namespace">
+<xacro:macro name="elbow_L_skin" params="parent namespace">
     <!-- Properties -->
     <xacro:property name="use_mesh_file" value="true" />
-    <xacro:property name="mesh_file" value="meshes/skin/elbow_R_skin.stl" />
+    <xacro:property name="mesh_file" value="meshes/skin/elbow_L_skin.stl" />
     <xacro:property name="mass" value="0.0" /> <!-- [kg] -->
     <xacro:property name="body_width" value="0.0" /> <!-- [m] -->

File: robots/h1-2/skin/shoulder_yaw_L_skin.xacro (robot description, xacro)
@@ -2,8 +2,8 @@
 <robot xmlns:xacro="http://ros.org/wiki/xacro">
 <!-- Macro definition for skin unit -->
-<xacro:macro name="shoulder_yaw_L_skin" params="parent namespace">
+<xacro:macro name="shoulder_yaw_R_skin" params="parent namespace">
     <!-- Properties -->
     <xacro:property name="use_mesh_file" value="true" />
-    <xacro:property name="mesh_file" value="meshes/skin/shoulder_yaw_L_skin.stl" />
+    <xacro:property name="mesh_file" value="meshes/skin/shoulder_yaw_R_skin.stl" />
     <xacro:property name="mass" value="0.0" /> <!-- [kg] -->
     <xacro:property name="body_width" value="0.0" /> <!-- [m] -->

File: robots/h1-2/skin/shoulder_yaw_R_skin.xacro (robot description, xacro)
@@ -2,8 +2,8 @@
 <robot xmlns:xacro="http://ros.org/wiki/xacro">
 <!-- Macro definition for skin unit -->
-<xacro:macro name="shoulder_yaw_R_skin" params="parent namespace">
+<xacro:macro name="shoulder_yaw_L_skin" params="parent namespace">
     <!-- Properties -->
     <xacro:property name="use_mesh_file" value="true" />
-    <xacro:property name="mesh_file" value="meshes/skin/shoulder_yaw_R_skin.stl" />
+    <xacro:property name="mesh_file" value="meshes/skin/shoulder_yaw_L_skin.stl" />
     <xacro:property name="mass" value="0.0" /> <!-- [kg] -->
     <xacro:property name="body_width" value="0.0" /> <!-- [m] -->
