Commit message: add tof clamps to link5_back skin

File: robots/h1-2/skin/shoulder_roll_R_skin.xacro (robot description, xacro)
@@ -30,8 +30,8 @@
         sensor_radius="${sensor_radius}"
         sensor_length="0.0"
-        normal_x="0.9815351963043213"
-        normal_y="-0.18700765073299408"
-        normal_z="-0.04020834341645241">
-        <origin xyz="0.02020913176238537 -0.010433539748191833 -0.1203891709446907" rpy="1.6110156774520874 -1.3015655042636354e-07 1.3825271129608154" />
+        normal_x="1.574"
+        normal_y="0.016"
+        normal_z="1.618">
+        <origin xyz="0.019 -0.001 0.022" rpy="-1.574 -0.072 -1.524" />
     </xacro:self_cap_sensor>
     <xacro:self_cap_sensor
@@ -41,8 +41,8 @@
         sensor_radius="${sensor_radius}"
         sensor_length="0.0"
-        normal_x="0.9996338486671448"
-        normal_y="0.013296284712851048"
-        normal_z="0.023566756397485733">
-        <origin xyz="0.02196035161614418 0.003525834996253252 0.006447893101722002" rpy="1.547227382659912 1.2260383641660155e-07 1.5840967893600464" />
+        normal_x="0.095"
+        normal_y="-1.642"
+        normal_z="-2.656">
+        <origin xyz="0.015 0.031 -0.046" rpy="-1.642 -0.107 -0.982" />
     </xacro:self_cap_sensor>
     <xacro:self_cap_sensor
@@ -52,8 +52,8 @@
         sensor_radius="${sensor_radius}"
         sensor_length="0.0"
-        normal_x="0.9888880252838135"
-        normal_y="-0.14034967124462128"
-        normal_z="-0.04901430755853653">
-        <origin xyz="0.021171631291508675 -0.013482555747032166 -0.03812651336193085" rpy="1.6198302507400513 3.5244884344365346e-08 1.4298112392425537" />
+        normal_x="-0.066"
+        normal_y="-1.636"
+        normal_z="2.606">
+        <origin xyz="0.013 -0.034 -0.049" rpy="1.637 -0.095 0.962" />
     </xacro:self_cap_sensor>
     <xacro:self_cap_sensor
@@ -63,8 +63,8 @@
         sensor_radius="${sensor_radius}"
         sensor_length="0.0"
-        normal_x="0.9694053530693054"
-        normal_y="-0.24535463750362396"
-        normal_z="-0.007379625923931599">
-        <origin xyz="0.019492628052830696 -0.013848518952727318 -0.07953478395938873" rpy="1.5781761407852173 -1.408326113505609e-07 1.3229039907455444" />
+        normal_x="1.561"
+        normal_y="-0.021"
+        normal_z="1.671">
+        <origin xyz="0.019 -0.000 -0.100" rpy="-1.561 0.100 -1.470" />
     </xacro:self_cap_sensor>
     <xacro:self_cap_sensor
@@ -74,8 +74,8 @@
         sensor_radius="${sensor_radius}"
         sensor_length="0.0"
-        normal_x="0.8133350610733032"
-        normal_y="0.5817909836769104"
-        normal_z="-0.002318537561222911">
-        <origin xyz="0.011047429405152798 0.03214484453201294 -0.08381814509630203" rpy="1.5731147527694702 -3.6292128413606406e-08 2.1917271614074707" />
+        normal_x="-1.566"
+        normal_y="-0.001"
+        normal_z="0.214">
+        <origin xyz="-0.039 0.052 -0.112" rpy="-1.566 -0.001 0.214" />
     </xacro:self_cap_sensor>
     <xacro:self_cap_sensor
@@ -85,30 +85,8 @@
         sensor_radius="${sensor_radius}"
         sensor_length="0.0"
-        normal_x="-0.9864919185638428"
-        normal_y="0.15094248950481415"
-        normal_z="-0.06364033371210098">
-        <origin xyz="-0.0885578915476799 0.008191447705030441 -0.12311510741710663" rpy="1.6344798803329468 4.719517221474234e-08 -1.7226282358169556" />
-    </xacro:self_cap_sensor>
-    <xacro:self_cap_sensor
-        robot_namespace="${namespace}"
-        parent="${namespace}_skin"
-        sensor_number="6"
-        sensor_radius="${sensor_radius}"
-        sensor_length="0.0"
-        normal_x="-0.1679488718509674"
-        normal_y="-0.9829021096229553"
-        normal_z="-0.07547598332166672">
-        <origin xyz="-0.043252378702163696 -0.05412545055150986 -0.12589296698570251" rpy="1.6463441848754883 -1.1537085065072006e-08 -0.16923603415489197" />
-    </xacro:self_cap_sensor>
-    <xacro:self_cap_sensor
-        robot_namespace="${namespace}"
-        parent="${namespace}_skin"
-        sensor_number="7"
-        sensor_radius="${sensor_radius}"
-        sensor_length="0.0"
-        normal_x="0.4207991361618042"
-        normal_y="0.9060245156288147"
-        normal_z="-0.04525141045451164">
-        <origin xyz="-0.010976525023579597 0.05005709081888199 -0.12077049911022186" rpy="1.6160632371902466 -1.495763335412903e-08 2.7067909240722656" />
+        normal_x="1.572"
+        normal_y="0.000"
+        normal_z="-0.184">
+        <origin xyz="-0.041 -0.052 -0.113" rpy="1.572 0.000 -0.184" />
     </xacro:self_cap_sensor>
     </xacro:macro>

File: robots/h1-2/skin/tof/shoulder_roll_R_skin.xacro (robot description, xacro)
@@ -5,5 +5,5 @@
     <!-- Properties -->
     <xacro:property name="use_mesh_file" value="true" />
-    <xacro:property name="mesh_file" value="package://gentact_descriptions_hybrid/robots/h1-2/meshes/skin/tof/shoulder_roll_R_skin.stl" />
+    <xacro:property name="mesh_file" value="meshes/skin/shoulder_roll_R_skin.stl" />
     <xacro:property name="mass" value="0.0" /> <!-- [kg] -->
     <xacro:property name="body_width" value="0.0" /> <!-- [m] -->
@@ -22,5 +22,5 @@
     use_mesh_file="${use_mesh_file}"
     mesh_file="${mesh_file}">
-    <origin xyz="-0.0342 0.2095 -0.43358" rpy="0 0 0" />
+    <origin xyz="0 0 0" rpy="0 0 0" />
     </xacro:dermis_base_macro>
     <xacro:self_cap_sensor
@@ -30,8 +30,8 @@
         sensor_radius="${sensor_radius}"
         sensor_length="0.0"
-        normal_x="0.977189"
-        normal_y="0.212370"
-        normal_z="0.001000">
-        <origin xyz="-0.033 0.049 -0.099" rpy="-1.566 -0.001 0.214" />
+        normal_x="1.574"
+        normal_y="0.016"
+        normal_z="1.618">
+        <origin xyz="0.019 -0.001 0.022" rpy="-1.574 -0.072 -1.524" />
     </xacro:self_cap_sensor>
     <xacro:self_cap_sensor
@@ -41,8 +41,8 @@
         sensor_radius="${sensor_radius}"
         sensor_length="0.0"
-        normal_x="0.991169"
-        normal_y="0.132608"
-        normal_z="-0.000000">
-        <origin xyz="-0.026 -0.049 -0.100" rpy="1.570 0.000 0.133" />
+        normal_x="0.095"
+        normal_y="-1.642"
+        normal_z="-2.656">
+        <origin xyz="0.015 0.031 -0.046" rpy="-1.642 -0.107 -0.982" />
     </xacro:self_cap_sensor>
     <xacro:self_cap_sensor
@@ -52,8 +52,8 @@
         sensor_radius="${sensor_radius}"
         sensor_length="0.0"
-        normal_x="0.046658"
-        normal_y="-0.996317"
-        normal_z="0.071938">
-        <origin xyz="0.017 -0.000 -0.028" rpy="-1.574 -0.072 -1.524" />
+        normal_x="-0.066"
+        normal_y="-1.636"
+        normal_z="2.606">
+        <origin xyz="0.013 -0.034 -0.049" rpy="1.637 -0.095 0.962" />
     </xacro:self_cap_sensor>
     <xacro:self_cap_sensor
@@ -63,8 +63,8 @@
         sensor_radius="${sensor_radius}"
         sensor_length="0.0"
-        normal_x="0.569302"
-        normal_y="0.816638"
-        normal_z="0.094857">
-        <origin xyz="0.012 -0.026 -0.091" rpy="1.637 -0.095 0.962" />
+        normal_x="1.561"
+        normal_y="-0.021"
+        normal_z="1.671">
+        <origin xyz="0.019 -0.000 -0.100" rpy="-1.561 0.100 -1.470" />
     </xacro:self_cap_sensor>
     <xacro:self_cap_sensor
@@ -74,8 +74,8 @@
         sensor_radius="${sensor_radius}"
         sensor_length="0.0"
-        normal_x="0.537327"
-        normal_y="-0.836837"
-        normal_z="0.104807">
-        <origin xyz="0.008 0.032 -0.085" rpy="-1.638 -0.105 -1.000" />
+        normal_x="-1.566"
+        normal_y="-0.001"
+        normal_z="0.214">
+        <origin xyz="-0.039 0.052 -0.112" rpy="-1.566 -0.001 0.214" />
     </xacro:self_cap_sensor>
     <xacro:self_cap_sensor
@@ -85,19 +85,8 @@
         sensor_radius="${sensor_radius}"
         sensor_length="0.0"
-        normal_x="0.537327"
-        normal_y="-0.836837"
-        normal_z="0.104807">
-        <origin xyz="0.013 -0.035 -0.006" rpy="1.637 -0.095 0.964" />
-    </xacro:self_cap_sensor>
-    <xacro:self_cap_sensor
-        robot_namespace="${namespace}"
-        parent="${namespace}_skin"
-        sensor_number="6"
-        sensor_radius="${sensor_radius}"
-        sensor_length="0.0"
-        normal_x="0.537327"
-        normal_y="-0.836837"
-        normal_z="0.104807">
-        <origin xyz="0.011 0.037 -0.002" rpy="-1.508 0.094 -0.984" />
+        normal_x="1.572"
+        normal_y="0.000"
+        normal_z="-0.184">
+        <origin xyz="-0.041 -0.052 -0.113" rpy="1.572 0.000 -0.184" />
     </xacro:self_cap_sensor>
     </xacro:macro>
