Commit message: added h1

File: robots/h1-2/h1_2_torso_skin.urdf (robot description, URDF)
Before this commit: robot h1_2, 103 links, 102 joints
Links:
- link head_skin: geometry visual mesh filename=meshes/skin/head_skin.stl scale=1 1 1
- link left_elbow_skin: geometry visual mesh filename=meshes/skin/elbow_L_skin.stl scale=1 1 1
- link left_shoulder_roll_skin: geometry visual mesh filename=meshes/skin/shoulder_roll_L_skin.stl scale=1 1 1
- link left_shoulder_yaw_skin: geometry visual mesh filename=meshes/skin/shoulder_yaw_L_skin.stl scale=1 1 1
- link right_elbow_skin: geometry visual mesh filename=meshes/skin/elbow_R_skin.stl scale=1 1 1
- link right_shoulder_roll_skin: geometry visual mesh filename=meshes/skin/shoulder_roll_R_skin.stl scale=1 1 1
- link right_shoulder_yaw_skin: geometry visual mesh filename=meshes/skin/shoulder_yaw_R_skin.stl scale=1 1 1
- link torso_skin: geometry visual mesh filename=meshes/skin/torso_skin.stl scale=1 1 1

File: robots/h1-2/skin/elbow_L_skin.xacro (robot description, xacro)
@@ -5,5 +5,5 @@
     <!-- Properties -->
     <xacro:property name="use_mesh_file" value="true" />
-    <xacro:property name="mesh_file" value="package://gentact_descriptions/h1-2/meshes/skin/elbow_L_skin.stl" />
+    <xacro:property name="mesh_file" value="meshes/skin/elbow_L_skin.stl" />
     <xacro:property name="mass" value="0.0" /> <!-- [kg] -->
     <xacro:property name="body_width" value="0.0" /> <!-- [m] -->

File: robots/h1-2/skin/elbow_R_skin.xacro (robot description, xacro)
@@ -5,5 +5,5 @@
     <!-- Properties -->
     <xacro:property name="use_mesh_file" value="true" />
-    <xacro:property name="mesh_file" value="package://gentact_descriptions/h1-2/meshes/skin/elbow_R_skin.stl" />
+    <xacro:property name="mesh_file" value="meshes/skin/elbow_R_skin.stl" />
     <xacro:property name="mass" value="0.0" /> <!-- [kg] -->
     <xacro:property name="body_width" value="0.0" /> <!-- [m] -->

File: robots/h1-2/skin/head_skin.xacro (robot description, xacro)
@@ -5,5 +5,5 @@
     <!-- Properties -->
     <xacro:property name="use_mesh_file" value="true" />
-    <xacro:property name="mesh_file" value="package://gentact_descriptions/h1-2/meshes/skin/head_skin.stl" />
+    <xacro:property name="mesh_file" value="meshes/skin/head_skin.stl" />
     <xacro:property name="mass" value="0.0" /> <!-- [kg] -->
     <xacro:property name="body_width" value="0.0" /> <!-- [m] -->

File: robots/h1-2/skin/shoulder_roll_L_skin.xacro (robot description, xacro)
@@ -5,5 +5,5 @@
     <!-- Properties -->
     <xacro:property name="use_mesh_file" value="true" />
-    <xacro:property name="mesh_file" value="package://gentact_descriptions/h1-2/meshes/skin/shoulder_roll_L_skin.stl" />
+    <xacro:property name="mesh_file" value="meshes/skin/shoulder_roll_L_skin.stl" />
     <xacro:property name="mass" value="0.0" /> <!-- [kg] -->
     <xacro:property name="body_width" value="0.0" /> <!-- [m] -->

File: robots/h1-2/skin/shoulder_roll_R_skin.xacro (robot description, xacro)
@@ -5,5 +5,5 @@
     <!-- Properties -->
     <xacro:property name="use_mesh_file" value="true" />
-    <xacro:property name="mesh_file" value="package://gentact_descriptions/h1-2/meshes/skin/shoulder_roll_R_skin.stl" />
+    <xacro:property name="mesh_file" value="meshes/skin/shoulder_roll_R_skin.stl" />
     <xacro:property name="mass" value="0.0" /> <!-- [kg] -->
     <xacro:property name="body_width" value="0.0" /> <!-- [m] -->

File: robots/h1-2/skin/shoulder_yaw_L_skin.xacro (robot description, xacro)
@@ -5,5 +5,5 @@
     <!-- Properties -->
     <xacro:property name="use_mesh_file" value="true" />
-    <xacro:property name="mesh_file" value="package://gentact_descriptions/h1-2/meshes/skin/shoulder_yaw_L_skin.stl" />
+    <xacro:property name="mesh_file" value="meshes/skin/shoulder_yaw_L_skin.stl" />
     <xacro:property name="mass" value="0.0" /> <!-- [kg] -->
     <xacro:property name="body_width" value="0.0" /> <!-- [m] -->

File: robots/h1-2/skin/shoulder_yaw_R_skin.xacro (robot description, xacro)
@@ -5,5 +5,5 @@
     <!-- Properties -->
     <xacro:property name="use_mesh_file" value="true" />
-    <xacro:property name="mesh_file" value="package://gentact_descriptions/h1-2/meshes/skin/shoulder_yaw_R_skin.stl" />
+    <xacro:property name="mesh_file" value="meshes/skin/shoulder_yaw_R_skin.stl" />
     <xacro:property name="mass" value="0.0" /> <!-- [kg] -->
     <xacro:property name="body_width" value="0.0" /> <!-- [m] -->

File: robots/h1-2/skin/torso_skin.xacro (robot description, xacro)
@@ -5,5 +5,5 @@
     <!-- Properties -->
     <xacro:property name="use_mesh_file" value="true" />
-    <xacro:property name="mesh_file" value="package://gentact_descriptions/h1-2/meshes/skin/torso_skin.stl" />
+    <xacro:property name="mesh_file" value="meshes/skin/torso_skin.stl" />
     <xacro:property name="mass" value="0.0" /> <!-- [kg] -->
     <xacro:property name="body_width" value="0.0" /> <!-- [m] -->

Commit message: added h1

File: robots/h1-2/h1_2_torso_skin.urdf (robot description, URDF)
Before this commit: robot h1_2, 103 links, 102 joints
Joints:
- joint head_base_joint: origin xyz=0 0 0 rpy=1.5707 0 0 -> xyz=0 0 0 rpy=0 0 0
- joint left_elbow_base_joint: origin xyz=0 0 0 rpy=1.5707 0 0 -> xyz=0 0 0 rpy=0 0 0
- joint left_shoulder_roll_base_joint: origin xyz=0 0 0 rpy=1.5707 0 0 -> xyz=0 0 0 rpy=0 0 0
- joint left_shoulder_yaw_base_joint: origin xyz=0 0 0 rpy=1.5707 0 0 -> xyz=0 0 0 rpy=0 0 0
- joint right_elbow_base_joint: origin xyz=0 0 0 rpy=1.5707 0 0 -> xyz=0 0 0 rpy=0 0 0
- joint right_shoulder_roll_base_joint: origin xyz=0 0 0 rpy=1.5707 0 0 -> xyz=0 0 0 rpy=0 0 0
- joint right_shoulder_yaw_base_joint: origin xyz=0 0 0 rpy=1.5707 0 0 -> xyz=0 0 0 rpy=0 0 0
- joint torso_base_joint: origin xyz=0 0 0 rpy=1.5707 0 0 -> xyz=0 0 0 rpy=0 0 0

File: robots/h1-2/skin/elbow_L_skin.xacro (robot description, xacro)
@@ -22,5 +22,5 @@
     use_mesh_file="${use_mesh_file}"
     mesh_file="${mesh_file}">
-    <origin xyz="0 0 0" rpy="1.5707 0 0" />
+    <origin xyz="0 0 0" rpy="0 0 0" />
     </xacro:dermis_base_macro>
     <xacro:self_cap_sensor

File: robots/h1-2/skin/elbow_R_skin.xacro (robot description, xacro)
@@ -22,5 +22,5 @@
     use_mesh_file="${use_mesh_file}"
     mesh_file="${mesh_file}">
-    <origin xyz="0 0 0" rpy="1.5707 0 0" />
+    <origin xyz="0 0 0" rpy="0 0 0" />
     </xacro:dermis_base_macro>
     <xacro:self_cap_sensor

File: robots/h1-2/skin/head_skin.xacro (robot description, xacro)
@@ -22,5 +22,5 @@
     use_mesh_file="${use_mesh_file}"
     mesh_file="${mesh_file}">
-    <origin xyz="0 0 0" rpy="1.5707 0 0" />
+    <origin xyz="0 0 0" rpy="0 0 0" />
     </xacro:dermis_base_macro>
     <xacro:self_cap_sensor

File: robots/h1-2/skin/shoulder_roll_L_skin.xacro (robot description, xacro)
@@ -22,5 +22,5 @@
     use_mesh_file="${use_mesh_file}"
     mesh_file="${mesh_file}">
-    <origin xyz="0 0 0" rpy="1.5707 0 0" />
+    <origin xyz="0 0 0" rpy="0 0 0" />
     </xacro:dermis_base_macro>
     <xacro:self_cap_sensor

File: robots/h1-2/skin/shoulder_roll_R_skin.xacro (robot description, xacro)
@@ -22,5 +22,5 @@
     use_mesh_file="${use_mesh_file}"
     mesh_file="${mesh_file}">
-    <origin xyz="0 0 0" rpy="1.5707 0 0" />
+    <origin xyz="0 0 0" rpy="0 0 0" />
     </xacro:dermis_base_macro>
     <xacro:self_cap_sensor

File: robots/h1-2/skin/shoulder_yaw_L_skin.xacro (robot description, xacro)
@@ -22,5 +22,5 @@
     use_mesh_file="${use_mesh_file}"
     mesh_file="${mesh_file}">
-    <origin xyz="0 0 0" rpy="1.5707 0 0" />
+    <origin xyz="0 0 0" rpy="0 0 0" />
     </xacro:dermis_base_macro>
     <xacro:self_cap_sensor

File: robots/h1-2/skin/shoulder_yaw_R_skin.xacro (robot description, xacro)
@@ -22,5 +22,5 @@
     use_mesh_file="${use_mesh_file}"
     mesh_file="${mesh_file}">
-    <origin xyz="0 0 0" rpy="1.5707 0 0" />
+    <origin xyz="0 0 0" rpy="0 0 0" />
     </xacro:dermis_base_macro>
     <xacro:self_cap_sensor

File: robots/h1-2/skin/torso_skin.xacro (robot description, xacro)
@@ -22,5 +22,5 @@
     use_mesh_file="${use_mesh_file}"
     mesh_file="${mesh_file}">
-    <origin xyz="0 0 0" rpy="1.5707 0 0" />
+    <origin xyz="0 0 0" rpy="0 0 0" />
     </xacro:dermis_base_macro>
     <xacro:self_cap_sensor
