Commit message: Fixed urdf

File: robots/h1-2/h1_2_torso_skin.urdf (robot description, URDF)
Before this commit: robot h1_2, 103 links, 102 joints
Links:
- removed link left_shoulder_roll_sensor_7
- added link left_elbow_sensor_10
- added link left_elbow_sensor_9
Joints:
- removed joint left_shoulder_roll_sensor_7_joint
- added joint left_elbow_sensor_10_joint: type fixed, parent left_elbow_skin, child left_elbow_sensor_10, origin xyz=-0.00305706518702209 0.01633271388709545 0.03314973786473274 rpy=1.3567856550216675 8.37537594833293e-09 -3.12361741065979, axis -0.017564237117767334 0.9770290851593018 0.21238082647323608
- added joint left_elbow_sensor_9_joint: type fixed, parent left_elbow_skin, child left_elbow_sensor_9, origin xyz=0.051280681043863297 0.013466577976942062 -0.010949196293950081 rpy=1.571230411529541 1.0519261905983512e-07 3.006434440612793, axis 0.1347469836473465 0.9908799529075623 -0.00043415927211754024
- joint left_elbow_sensor_0_joint: axis -0.0033466597087681293 -0.9991910457611084 -0.04007663577795029 -> 0.10508289933204651 0.932461142539978 0.34564992785453796; origin xyz=-0.0054705264046788216 -0.01703549548983574 -0.02506975084543228 rpy=1.6108835935592651 3.0750507695742613e-10 -0.003349356586113572 -> xyz=0.08154594898223877 0.008091652765870094 0.0070435362868011 rpy=1.2178651094436646 1.2016704964423752e-08 3.029371976852417
- joint left_elbow_sensor_1_joint: axis 0.03249296545982361 -0.9906070828437805 0.1328226923942566 -> 0.1332709938287735 0.9065275192260742 -0.4005580246448517; origin xyz=0.09776215255260468 -0.009773069061338902 -0.003952523693442345 rpy=1.4375799894332886 -2.939074983387968e-09 0.032789308577775955 -> xyz=0.03382901847362518 0.012922026216983795 -0.037048935890197754 rpy=-1.1586705446243286 -3.141592502593994 -0.14596709609031677
- joint left_elbow_sensor_2_joint: axis 0.13000711798667908 -0.9857586622238159 0.10666757822036743 -> 0.14815989136695862 0.8612227439880371 -0.4861522316932678; origin xyz=0.02981957234442234 -0.015662170946598053 0.0170421302318573 rpy=1.4639254808425903 -1.415918404745753e-08 0.13112856447696686 -> xyz=0.06889647245407104 0.006562706083059311 -0.03566919267177582 rpy=-1.063114881515503 -3.141592502593994 -0.17036668956279755
- joint left_elbow_sensor_3_joint: axis 0.12371029704809189 -0.8856444358825684 -0.4475819766521454 -> 0.000999619485810399 -0.28232553601264954 -0.9593181014060974; origin xyz=0.03183375298976898 -0.012470245361328125 -0.038558200001716614 rpy=2.034855842590332 1.6719945428178562e-09 0.1387859433889389 -> xyz=0.08601070940494537 -0.044811271131038666 -0.05210724472999573 rpy=2.8553733825683594 3.4038366569788536e-10 0.0035406488459557295
- joint left_elbow_sensor_4_joint: axis 0.06528738886117935 -0.5346206426620483 0.8425664901733398 -> 0.3274943232536316 0.8370455503463745 0.4382946193218231; origin xyz=0.09520145505666733 0.008756054565310478 0.02564341574907303 rpy=0.5687653422355652 -1.8162769066520923e-08 0.12151739746332169 -> xyz=0.041937582194805145 0.01046033576130867 0.024017266929149628 rpy=1.1170960664749146 8.192893119485234e-08 2.7686517238616943
- joint left_elbow_sensor_5_joint: axis 0.004111784510314465 -0.9999915361404419 2.02366391022224e-06 -> 0.040094517171382904 0.99919593334198 0.00014104926958680153; origin xyz=-0.006869952194392681 -0.017091382294893265 0.005429353564977646 rpy=1.5707944631576538 2.0792034760575007e-10 0.004111796617507935 -> xyz=0.021635523065924644 0.01642613485455513 0.00085951026994735 rpy=1.570655345916748 -1.6653562084911755e-08 3.101487398147583
- joint left_elbow_sensor_6_joint: axis 0.00975038856267929 0.10503476858139038 0.9944207668304443 -> 0.003345410106703639 0.9999943375587463 -0.0003027388593181968; origin xyz=0.08788560330867767 0.03748124837875366 0.03188776969909668 rpy=0.10568315535783768 -2.4437664336574016e-08 3.049027919769287 -> xyz=-0.007533484138548374 0.0170928705483675 -0.010090745985507965 rpy=1.571099042892456 -1.5052036062002117e-08 3.13824725151062
- joint left_elbow_sensor_7_joint: axis 0.049779538065195084 -0.26070669293403625 -0.9641338586807251 -> 0.06125080958008766 0.37824228405952454 -0.9236780405044556; origin xyz=0.08021856844425201 0.01752631552517414 -0.05247209593653679 rpy=2.8729567527770996 -1.6629815746682652e-08 0.188669815659523 -> xyz=0.08704763650894165 -0.014367843046784401 -0.05096221715211868 rpy=-0.39322516322135925 -3.1415927410125732 -0.160541832447052
- joint left_elbow_sensor_8_joint: axis 0.15267664194107056 -0.8526670932769775 -0.4996485412120819 -> 0.009998704306781292 -0.10753583163022995 0.9941509366035461; origin xyz=0.06785736232995987 -0.006429128348827362 -0.03632089123129845 rpy=2.093989372253418 -2.5215447507775934e-09 0.17718012630939484 -> xyz=0.08814304322004318 -0.03759463131427765 0.031867414712905884 rpy=0.10821068286895752 -5.978086470292965e-09 0.09271365404129028
- joint left_shoulder_roll_base_joint: origin xyz=0 0 0 rpy=0 0 0 -> xyz=0 0 0 rpy=0.0 0 0
- joint left_shoulder_roll_sensor_0_joint: axis 0.9815351963043213 -0.18700765073299408 -0.04020834341645241 -> 0.9997968077659607 -0.007021559402346611 0.018895627930760384; origin xyz=0.02020913176238537 -0.010433539748191833 -0.1203891709446907 rpy=1.6110156774520874 -1.3015655042636354e-07 1.3825271129608154 -> xyz=0.021975861862301826 -0.0021392295602709055 0.005330793093889952 rpy=1.551899790763855 -4.484040871943762e-08 1.563773512840271
- joint left_shoulder_roll_sensor_1_joint: axis 0.9996338486671448 0.013296284712851048 0.023566756397485733 -> 0.9265779256820679 0.37610265612602234 0.0003138364991173148; origin xyz=0.02196035161614418 0.003525834996253252 0.006447893101722002 rpy=1.547227382659912 1.2260383641660155e-07 1.5840967893600464 -> xyz=0.017285505309700966 0.021028343588113785 -0.09356498718261719 rpy=1.570482611656189 5.187961704677946e-08 1.9563831090927124
- joint left_shoulder_roll_sensor_2_joint: axis 0.9888880252838135 -0.14034967124462128 -0.04901430755853653 -> 0.9420590400695801 0.3258788585662842 -0.07954674959182739; origin xyz=0.021171631291508675 -0.013482555747032166 -0.03812651336193085 rpy=1.6198302507400513 3.5244884344365346e-08 1.4298112392425537 -> xyz=0.018528997898101807 0.021264299750328064 -0.05174817889928818 rpy=1.6504273414611816 -8.728313360961693e-08 1.9038336277008057
- joint left_shoulder_roll_sensor_3_joint: axis 0.9694053530693054 -0.24535463750362396 -0.007379625923931599 -> 0.9388141632080078 -0.3444167375564575 -0.002259491477161646; origin xyz=0.019492628052830696 -0.013848518952727318 -0.07953478395938873 rpy=1.5781761407852173 -1.408326113505609e-07 1.3229039907455444 -> xyz=0.017716117203235626 -0.019416000694036484 -0.09579524397850037 rpy=1.5730558633804321 2.0718655235896222e-08 1.2191780805587769
- joint left_shoulder_roll_sensor_4_joint: axis 0.8133350610733032 0.5817909836769104 -0.002318537561222911 -> 0.7647241353988647 -0.6394460201263428 -0.07940851151943207; origin xyz=0.011047429405152798 0.03214484453201294 -0.08381814509630203 rpy=1.5731147527694702 -3.6292128413606406e-08 2.1917271614074707 -> xyz=0.00962911918759346 -0.035556647926568985 -0.057738468050956726 rpy=1.6502885818481445 -9.019574775948058e-08 0.8743812441825867
- joint left_shoulder_roll_sensor_5_joint: axis -0.9864919185638428 0.15094248950481415 -0.06364033371210098 -> -0.1515629142522812 0.9850699305534363 -0.08164525777101517; origin xyz=-0.0885578915476799 0.008191447705030441 -0.12311510741710663 rpy=1.6344798803329468 4.719517221474234e-08 -1.7226282358169556 -> xyz=-0.042358122766017914 0.05419747531414032 -0.12676522135734558 rpy=1.6525324583053589 1.9534674322585488e-08 -2.9889297485351562
- joint left_shoulder_roll_sensor_6_joint: axis -0.1679488718509674 -0.9829021096229553 -0.07547598332166672 -> 0.4189722537994385 -0.906827986240387 -0.04610069841146469; origin xyz=-0.043252378702163696 -0.05412545055150986 -0.12589296698570251 rpy=1.6463441848754883 -1.1537085065072006e-08 -0.16923603415489197 -> xyz=-0.011077336966991425 -0.05010441690683365 -0.12087845802307129 rpy=1.6169135570526123 -2.047060831955605e-08 0.4328043460845947
- joint left_shoulder_yaw_sensor_0_joint: axis 0.9508576989173889 -0.12113388627767563 -0.28494971990585327 -> 0.9546116590499878 0.08776101469993591 -0.2846307158470154; origin xyz=0.04118751734495163 -0.004814512562006712 -0.08737954497337341 rpy=1.8597503900527954 1.1286831025358879e-08 1.4440847635269165 -> xyz=0.041529230773448944 0.003520205384120345 -0.08673007041215897 rpy=1.85941743850708 -4.787436225228703e-08 1.6624724864959717
- joint left_shoulder_yaw_sensor_1_joint: axis -0.6932508945465088 -0.7167385220527649 -0.07542620599269867 -> -0.6787640452384949 0.7300658226013184 -0.07926768064498901; origin xyz=-0.035796575248241425 -0.03355425223708153 -0.04064032435417175 rpy=1.646294355392456 1.8119585831755103e-09 -0.7687416672706604 -> xyz=-0.035132333636283875 0.03415091335773468 -0.04077912122011185 rpy=1.6501473188400269 6.971942667632902e-08 -2.3925929069519043
- joint left_shoulder_yaw_sensor_2_joint: axis 0.04019082337617874 -0.9604589939117432 -0.2755054235458374 -> -0.9902281165122986 0.13945573568344116 -0.0006956477300263941; origin xyz=0.0068807341158390045 -0.038329385221004486 -0.07258914411067963 rpy=1.8499118089675903 -2.4386073160798105e-09 0.04182104021310806 -> xyz=-0.04940275847911835 0.004836997017264366 -0.07897341996431351 rpy=1.5714919567108154 1.3637459517212847e-07 -1.7107082605361938
- joint left_shoulder_yaw_sensor_3_joint: axis -0.9944165349006653 -0.10552489757537842 -0.0004047837865073234 -> 0.033767059445381165 0.9608089327812195 -0.2751469612121582; origin xyz=-0.04953809827566147 -0.003564621554687619 -0.0796278566122055 rpy=1.571201205253601 3.790614400145387e-08 -1.4650746583938599 -> xyz=0.005767298396676779 0.03839176893234253 -0.07237497717142105 rpy=-1.2920538187026978 -3.1415927410125732 -0.03512994945049286
- joint left_shoulder_yaw_sensor_4_joint: axis -0.13521844148635864 0.9906842708587646 0.01614234782755375 -> -0.47221818566322327 -0.8795956969261169 0.05763210728764534; origin xyz=-0.00878828577697277 0.04951019585132599 -0.0318453386425972 rpy=1.5546531677246094 -2.4349319005523284e-08 -3.0059409141540527 -> xyz=-0.02568146213889122 -0.0444842129945755 -0.041484661400318146 rpy=1.5131322145462036 -1.965817375548795e-08 -0.492697536945343
- joint left_shoulder_yaw_sensor_5_joint: axis -0.16762951016426086 -0.9856319427490234 -0.020739588886499405 -> -0.1291467845439911 0.9913425445556641 -0.023686012253165245; origin xyz=-0.0280979685485363 -0.027626603841781616 -0.11977264285087585 rpy=1.5915374755859375 1.0039254760840777e-08 -0.16846124827861786 -> xyz=-0.02670200914144516 0.027768440544605255 -0.11980567127466202 rpy=1.594484806060791 -3.9004454777114006e-08 -3.01204776763916

File: robots/h1-2/skin/elbow_L_skin.xacro (robot description, xacro)
@@ -30,8 +30,8 @@
         sensor_radius="${sensor_radius}"
         sensor_length="0.0"
-        normal_x="-0.0033466597087681293"
-        normal_y="-0.9991910457611084"
-        normal_z="-0.04007663577795029">
-        <origin xyz="-0.0054705264046788216 -0.01703549548983574 -0.02506975084543228" rpy="1.6108835935592651 3.0750507695742613e-10 -0.003349356586113572" />
+        normal_x="0.10508289933204651"
+        normal_y="0.932461142539978"
+        normal_z="0.34564992785453796">
+        <origin xyz="0.08154594898223877 0.008091652765870094 0.0070435362868011" rpy="1.2178651094436646 1.2016704964423752e-08 3.029371976852417" />
     </xacro:self_cap_sensor>
     <xacro:self_cap_sensor
@@ -41,8 +41,8 @@
         sensor_radius="${sensor_radius}"
         sensor_length="0.0"
-        normal_x="0.03249296545982361"
-        normal_y="-0.9906070828437805"
-        normal_z="0.1328226923942566">
-        <origin xyz="0.09776215255260468 -0.009773069061338902 -0.003952523693442345" rpy="1.4375799894332886 -2.939074983387968e-09 0.032789308577775955" />
+        normal_x="0.1332709938287735"
+        normal_y="0.9065275192260742"
+        normal_z="-0.4005580246448517">
+        <origin xyz="0.03382901847362518 0.012922026216983795 -0.037048935890197754" rpy="-1.1586705446243286 -3.141592502593994 -0.14596709609031677" />
     </xacro:self_cap_sensor>
     <xacro:self_cap_sensor
@@ -52,8 +52,8 @@
         sensor_radius="${sensor_radius}"
         sensor_length="0.0"
-        normal_x="0.13000711798667908"
-        normal_y="-0.9857586622238159"
-        normal_z="0.10666757822036743">
-        <origin xyz="0.02981957234442234 -0.015662170946598053 0.0170421302318573" rpy="1.4639254808425903 -1.415918404745753e-08 0.13112856447696686" />
+        normal_x="0.14815989136695862"
+        normal_y="0.8612227439880371"
+        normal_z="-0.4861522316932678">
+        <origin xyz="0.06889647245407104 0.006562706083059311 -0.03566919267177582" rpy="-1.063114881515503 -3.141592502593994 -0.17036668956279755" />
     </xacro:self_cap_sensor>
     <xacro:self_cap_sensor
@@ -63,8 +63,8 @@
         sensor_radius="${sensor_radius}"
         sensor_length="0.0"
-        normal_x="0.12371029704809189"
-        normal_y="-0.8856444358825684"
-        normal_z="-0.4475819766521454">
-        <origin xyz="0.03183375298976898 -0.012470245361328125 -0.038558200001716614" rpy="2.034855842590332 1.6719945428178562e-09 0.1387859433889389" />
+        normal_x="0.000999619485810399"
+        normal_y="-0.28232553601264954"
+        normal_z="-0.9593181014060974">
+        <origin xyz="0.08601070940494537 -0.044811271131038666 -0.05210724472999573" rpy="2.8553733825683594 3.4038366569788536e-10 0.0035406488459557295" />
     </xacro:self_cap_sensor>
     <xacro:self_cap_sensor
@@ -74,8 +74,8 @@
         sensor_radius="${sensor_radius}"
         sensor_length="0.0"
-        normal_x="0.06528738886117935"
-        normal_y="-0.5346206426620483"
-        normal_z="0.8425664901733398">
-        <origin xyz="0.09520145505666733 0.008756054565310478 0.02564341574907303" rpy="0.5687653422355652 -1.8162769066520923e-08 0.12151739746332169" />
+        normal_x="0.3274943232536316"
+        normal_y="0.8370455503463745"
+        normal_z="0.4382946193218231">
+        <origin xyz="0.041937582194805145 0.01046033576130867 0.024017266929149628" rpy="1.1170960664749146 8.192893119485234e-08 2.7686517238616943" />
     </xacro:self_cap_sensor>
     <xacro:self_cap_sensor
@@ -85,8 +85,8 @@
         sensor_radius="${sensor_radius}"
         sensor_length="0.0"
-        normal_x="0.004111784510314465"
-        normal_y="-0.9999915361404419"
-        normal_z="2.02366391022224e-06">
-        <origin xyz="-0.006869952194392681 -0.017091382294893265 0.005429353564977646" rpy="1.5707944631576538 2.0792034760575007e-10 0.004111796617507935" />
+        normal_x="0.040094517171382904"
+        normal_y="0.99919593334198"
+        normal_z="0.00014104926958680153">
+        <origin xyz="0.021635523065924644 0.01642613485455513 0.00085951026994735" rpy="1.570655345916748 -1.6653562084911755e-08 3.101487398147583" />
     </xacro:self_cap_sensor>
     <xacro:self_cap_sensor
@@ -96,8 +96,8 @@
         sensor_radius="${sensor_radius}"
         sensor_length="0.0"
-        normal_x="0.00975038856267929"
-        normal_y="0.10503476858139038"
-        normal_z="0.9944207668304443">
-        <origin xyz="0.08788560330867767 0.03748124837875366 0.03188776969909668" rpy="0.10568315535783768 -2.4437664336574016e-08 3.049027919769287" />
+        normal_x="0.003345410106703639"
+        normal_y="0.9999943375587463"
+        normal_z="-0.0003027388593181968">
+        <origin xyz="-0.007533484138548374 0.0170928705483675 -0.010090745985507965" rpy="1.571099042892456 -1.5052036062002117e-08 3.13824725151062" />
     </xacro:self_cap_sensor>
     <xacro:self_cap_sensor
@@ -107,8 +107,8 @@
         sensor_radius="${sensor_radius}"
         sensor_length="0.0"
-        normal_x="0.049779538065195084"
-        normal_y="-0.26070669293403625"
-        normal_z="-0.9641338586807251">
-        <origin xyz="0.08021856844425201 0.01752631552517414 -0.05247209593653679" rpy="2.8729567527770996 -1.6629815746682652e-08 0.188669815659523" />
+        normal_x="0.06125080958008766"
+        normal_y="0.37824228405952454"
+        normal_z="-0.9236780405044556">
+        <origin xyz="0.08704763650894165 -0.014367843046784401 -0.05096221715211868" rpy="-0.39322516322135925 -3.1415927410125732 -0.160541832447052" />
     </xacro:self_cap_sensor>
     <xacro:self_cap_sensor
@@ -118,8 +118,30 @@
         sensor_radius="${sensor_radius}"
         sensor_length="0.0"
-        normal_x="0.15267664194107056"
-        normal_y="-0.8526670932769775"
-        normal_z="-0.4996485412120819">
-        <origin xyz="0.06785736232995987 -0.006429128348827362 -0.03632089123129845" rpy="2.093989372253418 -2.5215447507775934e-09 0.17718012630939484" />
+        normal_x="0.009998704306781292"
+        normal_y="-0.10753583163022995"
+        normal_z="0.9941509366035461">
+        <origin xyz="0.08814304322004318 -0.03759463131427765 0.031867414712905884" rpy="0.10821068286895752 -5.978086470292965e-09 0.09271365404129028" />
+    </xacro:self_cap_sensor>
+    <xacro:self_cap_sensor
+        robot_namespace="${namespace}"
+        parent="${namespace}_skin"
+        sensor_number="9"
+        sensor_radius="${sensor_radius}"
+        sensor_length="0.0"
+        normal_x="0.1347469836473465"
+        normal_y="0.9908799529075623"
+        normal_z="-0.00043415927211754024">
+        <origin xyz="0.051280681043863297 0.013466577976942062 -0.010949196293950081" rpy="1.571230411529541 1.0519261905983512e-07 3.006434440612793" />
+    </xacro:self_cap_sensor>
+    <xacro:self_cap_sensor
+        robot_namespace="${namespace}"
+        parent="${namespace}_skin"
+        sensor_number="10"
+        sensor_radius="${sensor_radius}"
+        sensor_length="0.0"
+        normal_x="-0.017564237117767334"
+        normal_y="0.9770290851593018"
+        normal_z="0.21238082647323608">
+        <origin xyz="-0.00305706518702209 0.01633271388709545 0.03314973786473274" rpy="1.3567856550216675 8.37537594833293e-09 -3.12361741065979" />
     </xacro:self_cap_sensor>
     </xacro:macro>
