Commit message: Fixed urdf

File: robots/h1-2/skin/shoulder_roll_L_skin.xacro (robot description, xacro)
@@ -22,5 +22,5 @@
     use_mesh_file="${use_mesh_file}"
     mesh_file="${mesh_file}">
-    <origin xyz="0 0 0" rpy="0 0 0" />
+    <origin xyz="0 0 0" rpy="0.0 0 0" />
     </xacro:dermis_base_macro>
     <xacro:self_cap_sensor
@@ -30,8 +30,8 @@
         sensor_radius="${sensor_radius}"
         sensor_length="0.0"
-        normal_x="0.9815351963043213"
-        normal_y="-0.18700765073299408"
-        normal_z="-0.04020834341645241">
-        <origin xyz="0.02020913176238537 -0.010433539748191833 -0.1203891709446907" rpy="1.6110156774520874 -1.3015655042636354e-07 1.3825271129608154" />
+        normal_x="0.9997968077659607"
+        normal_y="-0.007021559402346611"
+        normal_z="0.018895627930760384">
+        <origin xyz="0.021975861862301826 -0.0021392295602709055 0.005330793093889952" rpy="1.551899790763855 -4.484040871943762e-08 1.563773512840271" />
     </xacro:self_cap_sensor>
     <xacro:self_cap_sensor
@@ -41,8 +41,8 @@
         sensor_radius="${sensor_radius}"
         sensor_length="0.0"
-        normal_x="0.9996338486671448"
-        normal_y="0.013296284712851048"
-        normal_z="0.023566756397485733">
-        <origin xyz="0.02196035161614418 0.003525834996253252 0.006447893101722002" rpy="1.547227382659912 1.2260383641660155e-07 1.5840967893600464" />
+        normal_x="0.9265779256820679"
+        normal_y="0.37610265612602234"
+        normal_z="0.0003138364991173148">
+        <origin xyz="0.017285505309700966 0.021028343588113785 -0.09356498718261719" rpy="1.570482611656189 5.187961704677946e-08 1.9563831090927124" />
     </xacro:self_cap_sensor>
     <xacro:self_cap_sensor
@@ -52,8 +52,8 @@
         sensor_radius="${sensor_radius}"
         sensor_length="0.0"
-        normal_x="0.9888880252838135"
-        normal_y="-0.14034967124462128"
-        normal_z="-0.04901430755853653">
-        <origin xyz="0.021171631291508675 -0.013482555747032166 -0.03812651336193085" rpy="1.6198302507400513 3.5244884344365346e-08 1.4298112392425537" />
+        normal_x="0.9420590400695801"
+        normal_y="0.3258788585662842"
+        normal_z="-0.07954674959182739">
+        <origin xyz="0.018528997898101807 0.021264299750328064 -0.05174817889928818" rpy="1.6504273414611816 -8.728313360961693e-08 1.9038336277008057" />
     </xacro:self_cap_sensor>
     <xacro:self_cap_sensor
@@ -63,8 +63,8 @@
         sensor_radius="${sensor_radius}"
         sensor_length="0.0"
-        normal_x="0.9694053530693054"
-        normal_y="-0.24535463750362396"
-        normal_z="-0.007379625923931599">
-        <origin xyz="0.019492628052830696 -0.013848518952727318 -0.07953478395938873" rpy="1.5781761407852173 -1.408326113505609e-07 1.3229039907455444" />
+        normal_x="0.9388141632080078"
+        normal_y="-0.3444167375564575"
+        normal_z="-0.002259491477161646">
+        <origin xyz="0.017716117203235626 -0.019416000694036484 -0.09579524397850037" rpy="1.5730558633804321 2.0718655235896222e-08 1.2191780805587769" />
     </xacro:self_cap_sensor>
     <xacro:self_cap_sensor
@@ -74,8 +74,8 @@
         sensor_radius="${sensor_radius}"
         sensor_length="0.0"
-        normal_x="0.8133350610733032"
-        normal_y="0.5817909836769104"
-        normal_z="-0.002318537561222911">
-        <origin xyz="0.011047429405152798 0.03214484453201294 -0.08381814509630203" rpy="1.5731147527694702 -3.6292128413606406e-08 2.1917271614074707" />
+        normal_x="0.7647241353988647"
+        normal_y="-0.6394460201263428"
+        normal_z="-0.07940851151943207">
+        <origin xyz="0.00962911918759346 -0.035556647926568985 -0.057738468050956726" rpy="1.6502885818481445 -9.019574775948058e-08 0.8743812441825867" />
     </xacro:self_cap_sensor>
     <xacro:self_cap_sensor
@@ -85,8 +85,8 @@
         sensor_radius="${sensor_radius}"
         sensor_length="0.0"
-        normal_x="-0.9864919185638428"
-        normal_y="0.15094248950481415"
-        normal_z="-0.06364033371210098">
-        <origin xyz="-0.0885578915476799 0.008191447705030441 -0.12311510741710663" rpy="1.6344798803329468 4.719517221474234e-08 -1.7226282358169556" />
+        normal_x="-0.1515629142522812"
+        normal_y="0.9850699305534363"
+        normal_z="-0.08164525777101517">
+        <origin xyz="-0.042358122766017914 0.05419747531414032 -0.12676522135734558" rpy="1.6525324583053589 1.9534674322585488e-08 -2.9889297485351562" />
     </xacro:self_cap_sensor>
     <xacro:self_cap_sensor
@@ -96,19 +96,8 @@
         sensor_radius="${sensor_radius}"
         sensor_length="0.0"
-        normal_x="-0.1679488718509674"
-        normal_y="-0.9829021096229553"
-        normal_z="-0.07547598332166672">
-        <origin xyz="-0.043252378702163696 -0.05412545055150986 -0.12589296698570251" rpy="1.6463441848754883 -1.1537085065072006e-08 -0.16923603415489197" />
-    </xacro:self_cap_sensor>
-    <xacro:self_cap_sensor
-        robot_namespace="${namespace}"
-        parent="${namespace}_skin"
-        sensor_number="7"
-        sensor_radius="${sensor_radius}"
-        sensor_length="0.0"
-        normal_x="0.4207991361618042"
-        normal_y="0.9060245156288147"
-        normal_z="-0.04525141045451164">
-        <origin xyz="-0.010976525023579597 0.05005709081888199 -0.12077049911022186" rpy="1.6160632371902466 -1.495763335412903e-08 2.7067909240722656" />
+        normal_x="0.4189722537994385"
+        normal_y="-0.906827986240387"
+        normal_z="-0.04610069841146469">
+        <origin xyz="-0.011077336966991425 -0.05010441690683365 -0.12087845802307129" rpy="1.6169135570526123 -2.047060831955605e-08 0.4328043460845947" />
     </xacro:self_cap_sensor>
     </xacro:macro>

File: robots/h1-2/skin/shoulder_yaw_L_skin.xacro (robot description, xacro)
@@ -30,8 +30,8 @@
         sensor_radius="${sensor_radius}"
         sensor_length="0.0"
-        normal_x="0.9508576989173889"
-        normal_y="-0.12113388627767563"
-        normal_z="-0.28494971990585327">
-        <origin xyz="0.04118751734495163 -0.004814512562006712 -0.08737954497337341" rpy="1.8597503900527954 1.1286831025358879e-08 1.4440847635269165" />
+        normal_x="0.9546116590499878"
+        normal_y="0.08776101469993591"
+        normal_z="-0.2846307158470154">
+        <origin xyz="0.041529230773448944 0.003520205384120345 -0.08673007041215897" rpy="1.85941743850708 -4.787436225228703e-08 1.6624724864959717" />
     </xacro:self_cap_sensor>
     <xacro:self_cap_sensor
@@ -41,8 +41,8 @@
         sensor_radius="${sensor_radius}"
         sensor_length="0.0"
-        normal_x="-0.6932508945465088"
-        normal_y="-0.7167385220527649"
-        normal_z="-0.07542620599269867">
-        <origin xyz="-0.035796575248241425 -0.03355425223708153 -0.04064032435417175" rpy="1.646294355392456 1.8119585831755103e-09 -0.7687416672706604" />
+        normal_x="-0.6787640452384949"
+        normal_y="0.7300658226013184"
+        normal_z="-0.07926768064498901">
+        <origin xyz="-0.035132333636283875 0.03415091335773468 -0.04077912122011185" rpy="1.6501473188400269 6.971942667632902e-08 -2.3925929069519043" />
     </xacro:self_cap_sensor>
     <xacro:self_cap_sensor
@@ -52,8 +52,8 @@
         sensor_radius="${sensor_radius}"
         sensor_length="0.0"
-        normal_x="0.04019082337617874"
-        normal_y="-0.9604589939117432"
-        normal_z="-0.2755054235458374">
-        <origin xyz="0.0068807341158390045 -0.038329385221004486 -0.07258914411067963" rpy="1.8499118089675903 -2.4386073160798105e-09 0.04182104021310806" />
+        normal_x="-0.9902281165122986"
+        normal_y="0.13945573568344116"
+        normal_z="-0.0006956477300263941">
+        <origin xyz="-0.04940275847911835 0.004836997017264366 -0.07897341996431351" rpy="1.5714919567108154 1.3637459517212847e-07 -1.7107082605361938" />
     </xacro:self_cap_sensor>
     <xacro:self_cap_sensor
@@ -63,8 +63,8 @@
         sensor_radius="${sensor_radius}"
         sensor_length="0.0"
-        normal_x="-0.9944165349006653"
-        normal_y="-0.10552489757537842"
-        normal_z="-0.0004047837865073234">
-        <origin xyz="-0.04953809827566147 -0.003564621554687619 -0.0796278566122055" rpy="1.571201205253601 3.790614400145387e-08 -1.4650746583938599" />
+        normal_x="0.033767059445381165"
+        normal_y="0.9608089327812195"
+        normal_z="-0.2751469612121582">
+        <origin xyz="0.005767298396676779 0.03839176893234253 -0.07237497717142105" rpy="-1.2920538187026978 -3.1415927410125732 -0.03512994945049286" />
     </xacro:self_cap_sensor>
     <xacro:self_cap_sensor
@@ -74,8 +74,8 @@
         sensor_radius="${sensor_radius}"
         sensor_length="0.0"
-        normal_x="-0.13521844148635864"
-        normal_y="0.9906842708587646"
-        normal_z="0.01614234782755375">
-        <origin xyz="-0.00878828577697277 0.04951019585132599 -0.0318453386425972" rpy="1.5546531677246094 -2.4349319005523284e-08 -3.0059409141540527" />
+        normal_x="-0.47221818566322327"
+        normal_y="-0.8795956969261169"
+        normal_z="0.05763210728764534">
+        <origin xyz="-0.02568146213889122 -0.0444842129945755 -0.041484661400318146" rpy="1.5131322145462036 -1.965817375548795e-08 -0.492697536945343" />
     </xacro:self_cap_sensor>
     <xacro:self_cap_sensor
@@ -85,8 +85,8 @@
         sensor_radius="${sensor_radius}"
         sensor_length="0.0"
-        normal_x="-0.16762951016426086"
-        normal_y="-0.9856319427490234"
-        normal_z="-0.020739588886499405">
-        <origin xyz="-0.0280979685485363 -0.027626603841781616 -0.11977264285087585" rpy="1.5915374755859375 1.0039254760840777e-08 -0.16846124827861786" />
+        normal_x="-0.1291467845439911"
+        normal_y="0.9913425445556641"
+        normal_z="-0.023686012253165245">
+        <origin xyz="-0.02670200914144516 0.027768440544605255 -0.11980567127466202" rpy="1.594484806060791 -3.9004454777114006e-08 -3.01204776763916" />
     </xacro:self_cap_sensor>
     </xacro:macro>
