Commit message: add arg for output file

File: robots/h1-2/h1_2_handless_tof.xacro (robot description, xacro)
@@ -3,5 +3,5 @@
 <!-- xacro for ToF Skins made by Nick J. -->
   <!-- Properties -->
-  <xacro:property name="mesh_dir" value="meshes" />
+  <xacro:property name="mesh_dir" value="package://gentact_ros_tools_hybrid/meshes/h1_2" />
   <!-- Material colors -->
   <xacro:property name="material_grey" value="0.1 0.1 0.1 1" />
@@ -9,10 +9,10 @@
   <!-- Material macro -->
   <xacro:macro name="material_grey">
-    <material>
+    <material name="grey">
       <color rgba="${material_grey}"/>
     </material>
   </xacro:macro>
   <xacro:macro name="material_white">
-    <material>
+    <material name="white">
       <color rgba="${material_white}"/>
     </material>

File: robots/h1-2/skin/tof/shoulder_roll_R_skin.xacro (robot description, xacro)
@@ -22,5 +22,5 @@
     use_mesh_file="${use_mesh_file}"
     mesh_file="${mesh_file}">
-    <origin xyz="0 0 0" rpy="0 0 0" />
+    <origin xyz="-0.0342 0.2095 -0.43358" rpy="0 0 0" />
     </xacro:dermis_base_macro>
     <xacro:self_cap_sensor

Commit message: add h1_2 skins

File: robots/h1-2/h1_2_handless_tof.xacro (robot description, xacro)
@@ -494,6 +494,6 @@
     <limit lower="-0.95" upper="3.18" effort="18" velocity="20"/>
   </joint>
-  <!-- <xacro:include filename="./skin/elbow_L_skin.xacro" /> -->
-  <!-- <xacro:elbow_L_skin parent="left_elbow_link" namespace="left_elbow" /> -->
+  <xacro:include filename="./skin/tof/elbow_L_skin.xacro" />
+  <xacro:elbow_L_skin parent="left_elbow_link" namespace="left_elbow" />
   <link name="left_wrist_roll_link">
     <inertial>
@@ -660,6 +660,6 @@
     <limit lower="-3.01" upper="2.66" effort="18" velocity="20"/>
   </joint>
-  <!-- <xacro:include filename="./skin/shoulder_yaw_R_skin.xacro" /> -->
-  <!-- <xacro:shoulder_yaw_R_skin parent="right_shoulder_yaw_link" namespace="right_shoulder_yaw" /> -->
+  <xacro:include filename="./skin/tof/shoulder_yaw_R_skin.xacro" />
+  <xacro:shoulder_yaw_R_skin parent="right_shoulder_yaw_link" namespace="right_shoulder_yaw" />
   <link name="right_elbow_link">
     <inertial>
@@ -689,5 +689,5 @@
     <limit lower="-0.95" upper="3.18" effort="18" velocity="20"/>
   </joint>
-  <!-- <xacro:include filename="./skin/elbow_R_skin.xacro" /> -->
+  <!-- <xacro:include filename="./skin/tof/elbow_R_skin.xacro" /> -->
   <!-- <xacro:elbow_R_skin parent="right_elbow_link" namespace="right_elbow" /> -->
   <link name="right_wrist_roll_link">

File: robots/h1-2/skin/tof/shoulder_roll_R_skin.xacro (robot description, xacro)
@@ -5,5 +5,5 @@
     <!-- Properties -->
     <xacro:property name="use_mesh_file" value="true" />
-    <xacro:property name="mesh_file" value="meshes/skin/shoulder_roll_R_skin.stl" />
+    <xacro:property name="mesh_file" value="${mesh_dir}/skin/tof/shoulder_roll_R_skin.stl" />
     <xacro:property name="mass" value="0.0" /> <!-- [kg] -->
     <xacro:property name="body_width" value="0.0" /> <!-- [m] -->

Commit message: fixed link5 front and back skins

File: robots/h1-2/h1_2_handless_tof.xacro (robot description, xacro)
@@ -436,6 +436,6 @@
     <limit lower="-0.38" upper="3.4" effort="40" velocity="9"/>
   </joint>
-  <!-- <xacro:include filename="./skin/shoulder_roll_L_skin.xacro" /> -->
-  <!-- <xacro:shoulder_roll_L_skin parent="left_shoulder_roll_link" namespace="left_shoulder_roll" /> -->
+  <xacro:include filename="./skin/tof/shoulder_roll_L_skin.xacro" />
+  <xacro:shoulder_roll_L_skin parent="left_shoulder_roll_link" namespace="left_shoulder_roll" />
   <link name="left_shoulder_yaw_link">
     <inertial>

File: robots/h1-2/skin/tof/shoulder_roll_L_skin.xacro (robot description, xacro)
@@ -2,5 +2,5 @@
 <robot xmlns:xacro="http://ros.org/wiki/xacro">
 <!-- Macro definition for skin unit -->
-<xacro:macro name="shoulder_roll_R_skin" params="parent namespace">
+<xacro:macro name="shoulder_roll_L_skin" params="parent namespace">
     <!-- Properties -->
     <xacro:property name="use_mesh_file" value="true" />

File: robots/skin/hybrid/link3_hybrid.xacro (robot description, xacro)
@@ -26,21 +26,21 @@
     <!-- Instantiate sensors -->
     <xacro:self_cap_sensor robot_namespace="${namespace}" parent="${namespace}_skin" sensor_number="0"
-      sensor_radius="${sensor_radius}" sensor_length="${sensor_length}" normal_x="0" normal_y="0" normal_z="0">
+      sensor_radius="${sensor_radius}" sensor_length="${sensor_length}" normal_x="-0.46" normal_y="0.875" normal_z="0.151">
       <origin xyz="-0.025 0.052 -0.066" rpy="1.419 -0.000 -2.658" />
     </xacro:self_cap_sensor>
     <xacro:self_cap_sensor robot_namespace="${namespace}" parent="${namespace}_skin" sensor_number="1"
-      sensor_radius="${sensor_radius}" sensor_length="${sensor_length}" normal_x="0" normal_y="0" normal_z="0">
+      sensor_radius="${sensor_radius}" sensor_length="${sensor_length}" normal_x="-0.371" normal_y="0.89" normal_z="-0.264">
       <origin xyz="0.057 0.110 -0.019" rpy="1.838 -0.000 -2.747" />
     </xacro:self_cap_sensor>
     <xacro:self_cap_sensor robot_namespace="${namespace}" parent="${namespace}_skin" sensor_number="2"
-      sensor_radius="${sensor_radius}" sensor_length="${sensor_length}" normal_x="0" normal_y="0" normal_z="0">
+      sensor_radius="${sensor_radius}" sensor_length="${sensor_length}" normal_x="0.732" normal_y="0.662" normal_z="0.160">
       <origin xyz="0.124 0.101 0.009" rpy="1.410 0.000 2.306" />
     </xacro:self_cap_sensor>
     <xacro:self_cap_sensor robot_namespace="${namespace}" parent="${namespace}_skin" sensor_number="3"
-      sensor_radius="${sensor_radius}" sensor_length="${sensor_length}" normal_x="0" normal_y="0" normal_z="0">
+      sensor_radius="${sensor_radius}" sensor_length="${sensor_length}" normal_x="-0.885" normal_y="-0.441" normal_z="0.148">
       <origin xyz="-0.052 -0.026 -0.068" rpy="1.422 0.000 -1.108" />
     </xacro:self_cap_sensor>
     <xacro:self_cap_sensor robot_namespace="${namespace}" parent="${namespace}_skin" sensor_number="4"
-      sensor_radius="${sensor_radius}" sensor_length="${sensor_length}" normal_x="0" normal_y="0" normal_z="0">
+      sensor_radius="${sensor_radius}" sensor_length="${sensor_length}" normal_x="-0.689" normal_y="0.2" normal_z="0.697">
       <origin xyz="0.045 0.079 0.038" rpy="0.800 0.000 -1.854" />
     </xacro:self_cap_sensor>

File: robots/skin/hybrid/link5_hybrid_back.xacro (robot description, xacro)
@@ -1,9 +1,9 @@
 <?xml version="1.0"?>
 <robot xmlns:xacro="http://ros.org/wiki/xacro">
-  <!-- Macro definition for link5 pt 1 skin -->
+  <!-- Macro definition for link5 pt 2 skin -->
   <xacro:macro name="link5_back_skin" params="parent namespace">
     <!-- Properties -->
     <xacro:property name="use_mesh_file" value="true" />
-    <xacro:property name="mesh_file" value="package://gentact_descriptions_hybrid/meshes/skin/hybrid/link5_part1_hybrid_dermis.stl" />
+    <xacro:property name="mesh_file" value="package://gentact_descriptions_hybrid/meshes/skin/hybrid/link5_back_hybrid_dermis.stl" />
     <xacro:property name="mass" value="0.3" /> <!-- [kg] -->
     <xacro:property name="body_width" value="0.3" /> <!-- [m] -->
@@ -25,28 +25,20 @@
     </xacro:dermis_base_macro>
     <!-- Instantiate sensors -->
- <xacro:self_cap_sensor robot_namespace="${namespace}" parent="${namespace}_skin" sensor_number="0"
-      sensor_radius="${sensor_radius}" sensor_length="${sensor_length}" normal_x="-0.048" normal_y="0.984" normal_z="-0.173">
-      <origin xyz="-0.006 0.114 -0.097" rpy="-1.397 -3.142 0.049" />
+<xacro:self_cap_sensor robot_namespace="${namespace}" parent="${namespace}_skin" sensor_number="0"
+	    sensor_radius="${sensor_radius}" sensor_length="${sensor_length}" normal_x="-0.366" normal_y="-0.69" normal_z="0.625">
+    <origin xyz="-0.025 -0.042 -0.191" rpy="0.896 0.000 -0.487" />
     </xacro:self_cap_sensor>
     <xacro:self_cap_sensor robot_namespace="${namespace}" parent="${namespace}_skin" sensor_number="1"
-      sensor_radius="${sensor_radius}" sensor_length="${sensor_length}" normal_x="-0.374" normal_y="0.909" normal_z="-0.182">
-      <origin xyz="-0.021 0.102 -0.151" rpy="1.754 0.000 -2.751" />
+	    sensor_radius="${sensor_radius}" sensor_length="${sensor_length}" normal_x="-0.024" normal_y="-0.383" normal_z="0.923">
+    <origin xyz="-0.002 0.022 -0.152" rpy="0.394 0.000 -0.062" />
     </xacro:self_cap_sensor>
     <xacro:self_cap_sensor robot_namespace="${namespace}" parent="${namespace}_skin" sensor_number="2"
-      sensor_radius="${sensor_radius}" sensor_length="${sensor_length}" normal_x="-0.048" normal_y="0.972" normal_z="-0.232">
-      <origin xyz="-0.002 0.135 -0.018" rpy="-1.337 3.142 0.049" />
+	    sensor_radius="${sensor_radius}" sensor_length="${sensor_length}" normal_x="-0.028" normal_y="-0.982" normal_z="0.189">
+    <origin xyz="-0.000 0.058 -0.115" rpy="1.380 -0.000 -0.028" />
     </xacro:self_cap_sensor>
     <xacro:self_cap_sensor robot_namespace="${namespace}" parent="${namespace}_skin" sensor_number="3"
-      sensor_radius="${sensor_radius}" sensor_length="${sensor_length}" normal_x="0.376" normal_y="0.908" normal_z="-0.187">
-      <origin xyz="0.020 0.103 -0.148" rpy="1.758 -0.000 2.749" />
-    </xacro:self_cap_sensor>
-    <xacro:self_cap_sensor robot_namespace="${namespace}" parent="${namespace}_skin" sensor_number="4"
-      sensor_radius="${sensor_radius}" sensor_length="${sensor_length}" normal_x="0.864" normal_y="0.412" normal_z="0.289">
-      <origin xyz="0.049 0.108 0.014" rpy="1.278 0.000 2.016" />
-    </xacro:self_cap_sensor>
-    <xacro:self_cap_sensor robot_namespace="${namespace}" parent="${namespace}_skin" sensor_number="5"
-      sensor_radius="${sensor_radius}" sensor_length="${sensor_length}" normal_x="-0.865" normal_y="0.414" normal_z="0.285">
-      <origin xyz="-0.050 0.106 0.016" rpy="1.282 0.000 -2.017" />
+	    sensor_radius="${sensor_radius}" sensor_length="${sensor_length}" normal_x="0.377" normal_y="-0.687" normal_z="0.621">
+    <origin xyz="0.027 -0.041 -0.191" rpy="0.901 -0.000 0.501" />
     </xacro:self_cap_sensor>
   </xacro:macro>
-    </robot>
+   </robot>

File: robots/skin/hybrid/link5_hybrid_front.xacro (robot description, xacro)
@@ -1,9 +1,9 @@
 <?xml version="1.0"?>
 <robot xmlns:xacro="http://ros.org/wiki/xacro">
-  <!-- Macro definition for link5 pt 2 skin -->
+  <!-- Macro definition for link5 pt 1 skin -->
   <xacro:macro name="link5_front_skin" params="parent namespace">
     <!-- Properties -->
     <xacro:property name="use_mesh_file" value="true" />
-    <xacro:property name="mesh_file" value="package://gentact_descriptions_hybrid/meshes/skin/hybrid/link5_part2_hybrid_dermis.stl" />
+    <xacro:property name="mesh_file" value="package://gentact_descriptions_hybrid/meshes/skin/hybrid/link5_front_hybrid_dermis.stl" />
     <xacro:property name="mass" value="0.3" /> <!-- [kg] -->
     <xacro:property name="body_width" value="0.3" /> <!-- [m] -->
@@ -25,20 +25,28 @@
     </xacro:dermis_base_macro>
     <!-- Instantiate sensors -->
-<xacro:self_cap_sensor robot_namespace="${namespace}" parent="${namespace}_skin" sensor_number="0"
-	    sensor_radius="${sensor_radius}" sensor_length="${sensor_length}" normal_x="0" normal_y="0" normal_z="0">
-    <origin xyz="-0.025 -0.042 -0.191" rpy="0.896 0.000 -0.487" />
+ <xacro:self_cap_sensor robot_namespace="${namespace}" parent="${namespace}_skin" sensor_number="0"
+      sensor_radius="${sensor_radius}" sensor_length="${sensor_length}" normal_x="-0.048" normal_y="0.984" normal_z="-0.173">
+      <origin xyz="-0.006 0.114 -0.097" rpy="-1.397 -3.142 0.049" />
     </xacro:self_cap_sensor>
     <xacro:self_cap_sensor robot_namespace="${namespace}" parent="${namespace}_skin" sensor_number="1"
-	    sensor_radius="${sensor_radius}" sensor_length="${sensor_length}" normal_x="0" normal_y="0" normal_z="0">
-    <origin xyz="-0.002 0.022 -0.152" rpy="0.394 0.000 -0.062" />
+      sensor_radius="${sensor_radius}" sensor_length="${sensor_length}" normal_x="-0.374" normal_y="0.909" normal_z="-0.182">
+      <origin xyz="-0.021 0.102 -0.151" rpy="1.754 0.000 -2.751" />
     </xacro:self_cap_sensor>
     <xacro:self_cap_sensor robot_namespace="${namespace}" parent="${namespace}_skin" sensor_number="2"
-	    sensor_radius="${sensor_radius}" sensor_length="${sensor_length}" normal_x="0" normal_y="0" normal_z="0">
-    <origin xyz="-0.000 0.058 -0.115" rpy="1.380 -0.000 -0.028" />
+      sensor_radius="${sensor_radius}" sensor_length="${sensor_length}" normal_x="-0.048" normal_y="0.972" normal_z="-0.232">
+      <origin xyz="-0.002 0.135 -0.018" rpy="-1.337 3.142 0.049" />
     </xacro:self_cap_sensor>
     <xacro:self_cap_sensor robot_namespace="${namespace}" parent="${namespace}_skin" sensor_number="3"
-	    sensor_radius="${sensor_radius}" sensor_length="${sensor_length}" normal_x="0" normal_y="0" normal_z="0">
-    <origin xyz="0.027 -0.041 -0.191" rpy="0.901 -0.000 0.501" />
+      sensor_radius="${sensor_radius}" sensor_length="${sensor_length}" normal_x="0.376" normal_y="0.908" normal_z="-0.187">
+      <origin xyz="0.020 0.103 -0.148" rpy="1.758 -0.000 2.749" />
+    </xacro:self_cap_sensor>
+    <xacro:self_cap_sensor robot_namespace="${namespace}" parent="${namespace}_skin" sensor_number="4"
+      sensor_radius="${sensor_radius}" sensor_length="${sensor_length}" normal_x="0.864" normal_y="0.412" normal_z="0.289">
+      <origin xyz="0.049 0.108 0.014" rpy="1.278 0.000 2.016" />
+    </xacro:self_cap_sensor>
+    <xacro:self_cap_sensor robot_namespace="${namespace}" parent="${namespace}_skin" sensor_number="5"
+      sensor_radius="${sensor_radius}" sensor_length="${sensor_length}" normal_x="-0.865" normal_y="0.414" normal_z="0.285">
+      <origin xyz="-0.050 0.106 0.016" rpy="1.282 0.000 -2.017" />
     </xacro:self_cap_sensor>
   </xacro:macro>
-   </robot>
+    </robot>
