Commit message: Working sim

File: end_effectors/cobot_pump/cobot_pump.urdf.xacro (robot description, xacro)
@@ -1,11 +1,11 @@
 <?xml version="1.0" encoding="utf-8"?>
 <robot xmlns:xacro="http://www.ros.org/wiki/xacro" name="cobot_pump">
-  <xacro:include filename="$(find franka_description)/end_effectors/common/utils.xacro" />
-  <xacro:include filename="$(find franka_description)/end_effectors/common/ee_with_one_link.xacro"/>
-  <xacro:include filename="$(find franka_description)/end_effectors/cobot_pump/cobot_pump_arguments.xacro"/>
+  <xacro:include filename="$(find gentact_descriptions)/end_effectors/common/utils.xacro" />
+  <xacro:include filename="$(find gentact_descriptions)/end_effectors/common/ee_with_one_link.xacro"/>
+  <xacro:include filename="$(find gentact_descriptions)/end_effectors/cobot_pump/cobot_pump_arguments.xacro"/>
   <xacro:ee_with_one_link connected_to="$(arg special_connection)"
                           arm_id="$(arg arm_id)"
                           ee_id="$(arg ee_id)"
-                          ee_inertials="${xacro.load_yaml('$(find franka_description)/end_effectors/$(arg ee_id)/inertials.yaml')}"
+                          ee_inertials="${xacro.load_yaml('$(find gentact_descriptions)/end_effectors/$(arg ee_id)/inertials.yaml')}"
                           rpy_ee="$(arg rpy_ee)"
                           xyz_ee="$(arg xyz_ee)"

File: end_effectors/cobot_pump/cobot_pump_arguments.xacro (robot description, xacro)
@@ -22,4 +22,4 @@
   <xacro:arg name="gazebo" default="false" />
   <!-- Name of the description package -->
-  <xacro:arg name="description_pkg" default="franka_description" />
+  <xacro:arg name="description_pkg" default="gentact_descriptions" />
 </robot>

File: end_effectors/common/ee_with_one_link.xacro (robot description, xacro)
@@ -2,5 +2,5 @@
 <robot xmlns:xacro="http://www.ros.org/wiki/xacro" name="ee_with_one_link">
   <!-- safety_distance: Minimum safety distance in [m] by which the collision volumes are expanded and which is enforced during robot motions -->
-  <xacro:macro name="ee_with_one_link" params="connected_to:='' arm_id arm_prefix:='' ee_id ee_inertials rpy_ee:='0 0 0' xyz_ee:='0 0 0' tcp_xyz:='0 0 0' tcp_rpy:='0 0 0' safety_distance:=0 gazebo:=false description_pkg:=franka_description with_sc:=false">
+  <xacro:macro name="ee_with_one_link" params="connected_to:='' arm_id arm_prefix:='' ee_id ee_inertials rpy_ee:='0 0 0' xyz_ee:='0 0 0' tcp_xyz:='0 0 0' tcp_rpy:='0 0 0' safety_distance:=0 gazebo:=false description_pkg:=gentact_descriptions with_sc:=false">
     <xacro:property name="ee_prefix" default="robot_"/>
     <xacro:unless value="${arm_id == ''}">

File: end_effectors/common/franka_hand.xacro (robot description, xacro)
@@ -12,5 +12,5 @@
                        safety_distance:=0
                        gazebo:=false
-                       description_pkg:=franka_description
+                       description_pkg:=gentact_descriptions
                        with_sc:=false
                        no_prefix:=false">

File: end_effectors/common/utils.xacro (robot description, xacro)
@@ -42,5 +42,5 @@
       <collision name="${prefix}${name}_collision">
         <geometry>
-          <mesh filename="package://franka_description/meshes/robot_ee/${ee_id}/collision/${name}.stl" />
+          <mesh filename="package://gentact_descriptions/meshes/robot_ee/${ee_id}/collision/${name}.stl" />
         </geometry>
       </collision>

File: end_effectors/franka_hand/franka_hand_arguments.xacro (robot description, xacro)
@@ -24,4 +24,4 @@
   <xacro:arg name="gazebo" default="false" />
   <!-- Name of the description package -->
-  <xacro:arg name="description_pkg" default="franka_description" />
+  <xacro:arg name="description_pkg" default="gentact_descriptions" />
 </robot>

File: robots/common/franka_arm.ros2_control.xacro (robot description, xacro)
@@ -21,5 +21,5 @@
             <param name="state_following_offset">0.0</param>
           </xacro:if>
-          <xacro:if value="${gazebo and not (str(use_fake_hardware).lower() == 'true')}">
+          <xacro:if value="${gazebo}">
             <plugin>franka_ign_ros2_control/IgnitionSystem</plugin>
           </xacro:if>
@@ -86,5 +86,5 @@
       <xacro:general_purpose_io prefix="joint_4_sign" command_interface="elbow_command" index="1"/>
     </ros2_control>
-    <xacro:if value="${gazebo and not (str(use_fake_hardware).lower() == 'true')}">
+    <xacro:if value="${gazebo}">
       <gazebo>
         <plugin filename="franka_ign_ros2_control-system" name="ign_ros2_control::IgnitionROS2ControlPlugin">

File: robots/common/skin_unit_base.xacro (robot description, xacro)
@@ -33,14 +33,18 @@
     </joint>
     <link name="${robot_namespace}_sensor_${sensor_number}">
-      <visual>
-        <geometry>
-          <sphere radius="${sensor_radius}" /> <!-- [m] -->
-        </geometry>
-      </visual>
-      <collision>
-        <geometry>
-          <sphere radius="${sensor_radius}" /> <!-- [m] -->
-        </geometry>
-      </collision>
+      <xacro:if value="${sensor_radius > 0.0}">
+        <visual>
+          <geometry>
+            <sphere radius="${sensor_radius}" /> <!-- [m] -->
+          </geometry>
+        </visual>
+      </xacro:if>
+      <xacro:if value="${sensor_radius > 0.0}">
+        <collision>
+          <geometry>
+            <sphere radius="${sensor_radius}" /> <!-- [m] -->
+          </geometry>
+        </collision>
+      </xacro:if>
     </link>
   </xacro:macro>

File: urdf/compiled/fr3_full.urdf (robot description, URDF)
Before this commit: robot fr3, 54 links, 53 joints
Links:
- link fr3_hand: geometry collision mesh filename=package://gentact_descriptions/meshes/robot_ee/franka_hand_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; visual mesh filename=package://gentact_descriptions/meshes/robot_ee/franka_hand_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
