Commit message: added link2 correct orientation

File: end_effectors/cobot_pump/cobot_pump.urdf.xacro (robot description, xacro)
@@ -1,11 +1,11 @@
 <?xml version="1.0" encoding="utf-8"?>
 <robot xmlns:xacro="http://www.ros.org/wiki/xacro" name="cobot_pump">
-  <xacro:include filename="$(find gentact_descriptions)/end_effectors/common/utils.xacro" />
-  <xacro:include filename="$(find gentact_descriptions)/end_effectors/common/ee_with_one_link.xacro"/>
-  <xacro:include filename="$(find gentact_descriptions)/end_effectors/cobot_pump/cobot_pump_arguments.xacro"/>
+  <xacro:include filename="$(find gentact_descriptions_hybrid)/end_effectors/common/utils.xacro" />
+  <xacro:include filename="$(find gentact_descriptions_hybrid)/end_effectors/common/ee_with_one_link.xacro"/>
+  <xacro:include filename="$(find gentact_descriptions_hybrid)/end_effectors/cobot_pump/cobot_pump_arguments.xacro"/>
   <xacro:ee_with_one_link connected_to="$(arg special_connection)"
                           arm_id="$(arg arm_id)"
                           ee_id="$(arg ee_id)"
-                          ee_inertials="${xacro.load_yaml('$(find gentact_descriptions)/end_effectors/$(arg ee_id)/inertials.yaml')}"
+                          ee_inertials="${xacro.load_yaml('$(find gentact_descriptions_hybrid)/end_effectors/$(arg ee_id)/inertials.yaml')}"
                           rpy_ee="$(arg rpy_ee)"
                           xyz_ee="$(arg xyz_ee)"

File: end_effectors/cobot_pump/cobot_pump_arguments.xacro (robot description, xacro)
@@ -22,4 +22,4 @@
   <xacro:arg name="gazebo" default="false" />
   <!-- Name of the description package -->
-  <xacro:arg name="description_pkg" default="gentact_descriptions" />
+  <xacro:arg name="description_pkg" default="gentact_descriptions_hybrid" />
 </robot>

File: end_effectors/common/ee_with_one_link.xacro (robot description, xacro)
@@ -2,5 +2,5 @@
 <robot xmlns:xacro="http://www.ros.org/wiki/xacro" name="ee_with_one_link">
   <!-- safety_distance: Minimum safety distance in [m] by which the collision volumes are expanded and which is enforced during robot motions -->
-  <xacro:macro name="ee_with_one_link" params="connected_to:='' arm_id arm_prefix:='' ee_id ee_inertials rpy_ee:='0 0 0' xyz_ee:='0 0 0' tcp_xyz:='0 0 0' tcp_rpy:='0 0 0' safety_distance:=0 gazebo:=false description_pkg:=gentact_descriptions with_sc:=false">
+  <xacro:macro name="ee_with_one_link" params="connected_to:='' arm_id arm_prefix:='' ee_id ee_inertials rpy_ee:='0 0 0' xyz_ee:='0 0 0' tcp_xyz:='0 0 0' tcp_rpy:='0 0 0' safety_distance:=0 gazebo:=false description_pkg:=gentact_descriptions_hybrid with_sc:=false">
     <xacro:property name="ee_prefix" default="robot_"/>
     <xacro:unless value="${arm_id == ''}">

File: end_effectors/common/franka_hand.xacro (robot description, xacro)
@@ -12,5 +12,5 @@
                        safety_distance:=0
                        gazebo:=false
-                       description_pkg:=gentact_descriptions
+                       description_pkg:=gentact_descriptions_hybrid
                        with_sc:=false
                        no_prefix:=false">

File: end_effectors/common/utils.xacro (robot description, xacro)
@@ -42,5 +42,5 @@
       <collision name="${prefix}${name}_collision">
         <geometry>
-          <mesh filename="package://gentact_descriptions/meshes/robot_ee/${ee_id}/collision/${name}.stl" />
+          <mesh filename="package://gentact_descriptions_hybrid/meshes/robot_ee/${ee_id}/collision/${name}.stl" />
         </geometry>
       </collision>

File: end_effectors/franka_hand/franka_hand_arguments.xacro (robot description, xacro)
@@ -24,4 +24,4 @@
   <xacro:arg name="gazebo" default="false" />
   <!-- Name of the description package -->
-  <xacro:arg name="description_pkg" default="gentact_descriptions" />
+  <xacro:arg name="description_pkg" default="gentact_descriptions_hybrid" />
 </robot>

File: robots/common/franka_arm.xacro (robot description, xacro)
@@ -1,13 +1,13 @@
 <?xml version='1.0' encoding='utf-8'?>
 <robot xmlns:xacro="http://www.ros.org/wiki/xacro" name="franka_arm">
-  <xacro:include filename="$(find gentact_descriptions)/robots/common/utils.xacro" />
-  <xacro:include filename="$(find gentact_descriptions)/robots/common/skin_unit_base.xacro" />
+  <xacro:include filename="$(find gentact_descriptions_hybrid)/robots/common/utils.xacro" />
+  <xacro:include filename="$(find gentact_descriptions_hybrid)/robots/common/skin_unit_base.xacro" />
   <!-- safety_distance: Minimum safety distance in [m] by which the collision volumes are expanded and which is enforced during robot motions -->
   <!-- arm_id: Namespace of the robot arm. Serves to differentiate between arms in case of multiple instances. -->
-  <!-- joint_limits: description of the joint limits that comes from a YAML file. Example definition: ${xacro.load_yaml('$(find gentact_descriptions)/robots/fr3/joint_limits.yaml')} -->
-  <!-- kinematics: description of the kinematics that comes from a YAML file. Example definition: ${xacro.load_yaml('$(find gentact_descriptions)/robots/fr3/kinematics.yaml')} -->
-  <!-- inertials: description of the inertials that comes from a YAML file. Example definition: ${xacro.load_yaml('$(find gentact_descriptions)/robots/fr3/inertials.yaml')} -->
-  <!-- dynamics: description of the dynamics that comes from a YAML file. Example definition: ${xacro.load_yaml('$(find gentact_descriptions)/robots/fr3/dynamics.yaml')} -->
-  <xacro:macro name="franka_arm" params="arm_id arm_prefix:='' no_prefix:=false description_pkg:='gentact_descriptions' connected_to:='base' xyz:='0 0 0' rpy:='0 0 0' gazebo:='false' safety_distance:=0 joint_limits inertials kinematics dynamics with_sc:=false, link1_skin:='' link2_skin:='' link3_skin:='' link4_skin:='' link5_front_skin:='' link5_back_skin:='' link6_skin:=''">
+  <!-- joint_limits: description of the joint limits that comes from a YAML file. Example definition: ${xacro.load_yaml('$(find gentact_descriptions_hybrid)/robots/fr3/joint_limits.yaml')} -->
+  <!-- kinematics: description of the kinematics that comes from a YAML file. Example definition: ${xacro.load_yaml('$(find gentact_descriptions_hybrid)/robots/fr3/kinematics.yaml')} -->
+  <!-- inertials: description of the inertials that comes from a YAML file. Example definition: ${xacro.load_yaml('$(find gentact_descriptions_hybrid)/robots/fr3/inertials.yaml')} -->
+  <!-- dynamics: description of the dynamics that comes from a YAML file. Example definition: ${xacro.load_yaml('$(find gentact_descriptions_hybrid)/robots/fr3/dynamics.yaml')} -->
+  <xacro:macro name="franka_arm" params="arm_id arm_prefix:='' no_prefix:=false description_pkg:='gentact_descriptions_hybrid' connected_to:='base' xyz:='0 0 0' rpy:='0 0 0' gazebo:='false' safety_distance:=0 joint_limits inertials kinematics dynamics with_sc:=false, link1_skin:='' link2_skin:='' link3_skin:='' link4_skin:='' link5_front_skin:='' link5_back_skin:='' link6_skin:=''">
     <!-- Define a property that defaults to 'arm_prefix_arm_id' concatenated with an underscore if 'no_prefix' is not set -->
     <xacro:property name="prefix" value="${'' if no_prefix else arm_prefix + arm_id + '_'}" />

File: robots/common/franka_robot _hybrid.xacro (robot description, xacro)
@@ -27,5 +27,5 @@
                       no_prefix:='false'
                       arm_prefix:=''
-                      description_pkg:='gentact_descriptions'
+                      description_pkg:='gentact_descriptions_hybrid'
                       connected_to:='base'
                       link1_skin:=''
@@ -36,6 +36,6 @@
                       link5_back_skin:=''
                       link6_skin:=''">
-    <xacro:include filename="$(find gentact_descriptions)/robots/common/utils.xacro" />
-    <xacro:include filename="$(find gentact_descriptions)/robots/common/franka_arm.xacro" />
+    <xacro:include filename="$(find gentact_descriptions_hybrid)/robots/common/utils.xacro" />
+    <xacro:include filename="$(find gentact_descriptions_hybrid)/robots/common/franka_arm.xacro" />
     <xacro:franka_arm
       arm_id="${arm_id}"
@@ -61,6 +61,6 @@
     />
     <xacro:if value="${hand and ee_id == 'franka_hand'}">
-      <xacro:include filename="$(find gentact_descriptions)/end_effectors/common/franka_hand.xacro"/>
-      <xacro:include filename="$(find gentact_descriptions)/end_effectors/common/utils.xacro" />
+      <xacro:include filename="$(find gentact_descriptions_hybrid)/end_effectors/common/franka_hand.xacro"/>
+      <xacro:include filename="$(find gentact_descriptions_hybrid)/end_effectors/common/utils.xacro" />
       <xacro:if value="${arm_id == 'fp3'}">
         <xacro:property name="ee_color" value="black" />
@@ -76,5 +76,5 @@
         arm_prefix="${arm_prefix}"
         ee_id="${ee_id}_${ee_color}"
-        ee_inertials="${xacro.load_yaml('$(find gentact_descriptions)/end_effectors/' + ee_id + '/inertials.yaml')}"
+        ee_inertials="${xacro.load_yaml('$(find gentact_descriptions_hybrid)/end_effectors/' + ee_id + '/inertials.yaml')}"
         rpy_ee="${rpy_ee}"
         xyz_ee="${xyz_ee}"
@@ -88,6 +88,6 @@
     </xacro:if>
     <xacro:if value="${hand and ee_id != 'none' and ee_id != 'franka_hand'}">
-      <xacro:include filename="$(find gentact_descriptions)/end_effectors/common/ee_with_one_link.xacro"/>
-      <xacro:include filename="$(find gentact_descriptions)/end_effectors/common/utils.xacro" />
+      <xacro:include filename="$(find gentact_descriptions_hybrid)/end_effectors/common/ee_with_one_link.xacro"/>
+      <xacro:include filename="$(find gentact_descriptions_hybrid)/end_effectors/common/utils.xacro" />
       <xacro:property name="special_connection" value="${special_connection}" />
       <xacro:property name="connection" value="${special_connection if special_connection == '' else arm_id + '_link8'}" />
@@ -97,5 +97,5 @@
         arm_prefix="${arm_prefix}"
         ee_id="${ee_id}"
-        ee_inertials="${xacro.load_yaml('$(find gentact_descriptions)/end_effectors/${ee_id}/inertials.yaml')}"
+        ee_inertials="${xacro.load_yaml('$(find gentact_descriptions_hybrid)/end_effectors/${ee_id}/inertials.yaml')}"
         rpy_ee="${rpy_ee}"
         xyz_ee="${xyz_ee}"
@@ -156,5 +156,5 @@
     </xacro:if>
     <xacro:if value="${ros2_control}">
-      <xacro:include filename="$(find gentact_descriptions)/robots/common/franka_arm.ros2_control.xacro"/>
+      <xacro:include filename="$(find gentact_descriptions_hybrid)/robots/common/franka_arm.ros2_control.xacro"/>
       <xacro:franka_arm_ros2_control
           arm_id="${arm_id}"

File: robots/fr3/fr3.urdf.xacro (robot description, xacro)
@@ -1,5 +1,5 @@
 <?xml version='1.0' encoding='utf-8'?>
 <robot xmlns:xacro="http://www.ros.org/wiki/xacro" name="fr3">
-  <xacro:include filename="$(find gentact_descriptions)/robots/common/franka_robot.xacro"/>
+  <xacro:include filename="$(find gentact_descriptions_hybrid)/robots/common/franka_robot.xacro"/>
   <!--
     DEPRECATION NOTICE
@@ -43,13 +43,13 @@
   <xacro:arg name="gazebo_effort" default="false" />
   <!-- Name of the description package -->
-  <xacro:arg name="description_pkg" default="gentact_descriptions" />
+  <xacro:arg name="description_pkg" default="gentact_descriptions_hybrid" />
   <!-- Append an underscore to the user-provided prefix, if non-empty. -->
   <xacro:property name="prefix" value="$(arg arm_prefix)"/>
   <xacro:property name="modified_prefix" value="${prefix + '_' if prefix else ''}"/>
   <xacro:franka_robot arm_id="fr3"
-                      joint_limits="${xacro.load_yaml('$(find gentact_descriptions)/robots/fr3/joint_limits.yaml')}"
-                      inertials="${xacro.load_yaml('$(find gentact_descriptions)/robots/fr3/inertials.yaml')}"
-                      kinematics="${xacro.load_yaml('$(find gentact_descriptions)/robots/fr3/kinematics.yaml')}"
-                      dynamics="${xacro.load_yaml('$(find gentact_descriptions)/robots/fr3/dynamics.yaml')}"
+                      joint_limits="${xacro.load_yaml('$(find gentact_descriptions_hybrid)/robots/fr3/joint_limits.yaml')}"
+                      inertials="${xacro.load_yaml('$(find gentact_descriptions_hybrid)/robots/fr3/inertials.yaml')}"
+                      kinematics="${xacro.load_yaml('$(find gentact_descriptions_hybrid)/robots/fr3/kinematics.yaml')}"
+                      dynamics="${xacro.load_yaml('$(find gentact_descriptions_hybrid)/robots/fr3/dynamics.yaml')}"
                       gazebo="$(arg gazebo)"
                       hand="$(arg hand)"

File: robots/fr3/fr3_full_skin.urdf.xacro (robot description, xacro)
@@ -1,5 +1,5 @@
 <?xml version='1.0' encoding='utf-8'?>
 <robot xmlns:xacro="http://www.ros.org/wiki/xacro" name="fr3">
-  <xacro:include filename="$(find gentact_descriptions)/robots/common/franka_robot.xacro"/>
+  <xacro:include filename="$(find gentact_descriptions_hybrid)/robots/common/franka_robot.xacro"/>
   <!--
     DEPRECATION NOTICE
@@ -43,5 +43,5 @@
   <xacro:arg name="gazebo_effort" default="false" />
   <!-- Name of the description package -->
-  <xacro:arg name="description_pkg" default="gentact_descriptions" />
+  <xacro:arg name="description_pkg" default="gentact_descriptions_hybrid" />
   <!-- Define arguments for skin configurations -->
   <xacro:arg name="link1_skin" default=""/>
@@ -56,8 +56,8 @@
   <xacro:property name="modified_prefix" value="${prefix + '_' if prefix else ''}"/>
   <xacro:franka_robot arm_id="fr3"
-                      joint_limits="${xacro.load_yaml('$(find gentact_descriptions)/robots/fr3/joint_limits.yaml')}"
-                      inertials="${xacro.load_yaml('$(find gentact_descriptions)/robots/fr3/inertials.yaml')}"
-                      kinematics="${xacro.load_yaml('$(find gentact_descriptions)/robots/fr3/kinematics.yaml')}"
-                      dynamics="${xacro.load_yaml('$(find gentact_descriptions)/robots/fr3/dynamics.yaml')}"
+                      joint_limits="${xacro.load_yaml('$(find gentact_descriptions_hybrid)/robots/fr3/joint_limits.yaml')}"
+                      inertials="${xacro.load_yaml('$(find gentact_descriptions_hybrid)/robots/fr3/inertials.yaml')}"
+                      kinematics="${xacro.load_yaml('$(find gentact_descriptions_hybrid)/robots/fr3/kinematics.yaml')}"
+                      dynamics="${xacro.load_yaml('$(find gentact_descriptions_hybrid)/robots/fr3/dynamics.yaml')}"
                       gazebo="$(arg gazebo)"
                       hand="$(arg hand)"

File: robots/h1-2/skin/elbow_L_skin.xacro (robot description, xacro)
@@ -12,5 +12,5 @@
     <xacro:property name="sensor_radius" value="0.0" /> <!-- [m] -->
     <!-- Included URDF Files (NEEDED FOR BASE SKIN UNIT) -->
-    <xacro:include filename="$(find gentact_descriptions)/robots/common/skin_unit_base.xacro" />
+    <xacro:include filename="$(find gentact_descriptions_hybrid)/robots/common/skin_unit_base.xacro" />
     <!-- Instantiate dermis once -->
     <xacro:dermis_base_macro

File: robots/h1-2/skin/elbow_R_skin.xacro (robot description, xacro)
@@ -12,5 +12,5 @@
     <xacro:property name="sensor_radius" value="0.0" /> <!-- [m] -->
     <!-- Included URDF Files (NEEDED FOR BASE SKIN UNIT) -->
-    <xacro:include filename="$(find gentact_descriptions)/robots/common/skin_unit_base.xacro" />
+    <xacro:include filename="$(find gentact_descriptions_hybrid)/robots/common/skin_unit_base.xacro" />
     <!-- Instantiate dermis once -->
     <xacro:dermis_base_macro

File: robots/h1-2/skin/head_skin.xacro (robot description, xacro)
@@ -12,5 +12,5 @@
     <xacro:property name="sensor_radius" value="0.0" /> <!-- [m] -->
     <!-- Included URDF Files (NEEDED FOR BASE SKIN UNIT) -->
-    <xacro:include filename="$(find gentact_descriptions)/robots/common/skin_unit_base.xacro" />
+    <xacro:include filename="$(find gentact_descriptions_hybrid)/robots/common/skin_unit_base.xacro" />
     <!-- Instantiate dermis once -->
     <xacro:dermis_base_macro

File: robots/h1-2/skin/right_shoulder_roll_skin.xacro (robot description, xacro)
@@ -12,5 +12,5 @@
     <xacro:property name="sensor_radius" value="0.0" /> <!-- [m] -->
     <!-- Included URDF Files (NEEDED FOR BASE SKIN UNIT) -->
-    <xacro:include filename="$(find gentact_descriptions)/robots/common/skin_unit_base.xacro" />
+    <xacro:include filename="$(find gentact_descriptions_hybrid)/robots/common/skin_unit_base.xacro" />
     <!-- Instantiate dermis once -->
     <xacro:dermis_base_macro

File: robots/h1-2/skin/shoulder_roll_L_skin.xacro (robot description, xacro)
@@ -12,5 +12,5 @@
     <xacro:property name="sensor_radius" value="0.0" /> <!-- [m] -->
     <!-- Included URDF Files (NEEDED FOR BASE SKIN UNIT) -->
-    <xacro:include filename="$(find gentact_descriptions)/robots/common/skin_unit_base.xacro" />
+    <xacro:include filename="$(find gentact_descriptions_hybrid)/robots/common/skin_unit_base.xacro" />
     <!-- Instantiate dermis once -->
     <xacro:dermis_base_macro

File: robots/h1-2/skin/shoulder_roll_R_skin.xacro (robot description, xacro)
@@ -12,5 +12,5 @@
     <xacro:property name="sensor_radius" value="0.0" /> <!-- [m] -->
     <!-- Included URDF Files (NEEDED FOR BASE SKIN UNIT) -->
-    <xacro:include filename="$(find gentact_descriptions)/robots/common/skin_unit_base.xacro" />
+    <xacro:include filename="$(find gentact_descriptions_hybrid)/robots/common/skin_unit_base.xacro" />
     <!-- Instantiate dermis once -->
     <xacro:dermis_base_macro

File: robots/h1-2/skin/shoulder_yaw_L_skin.xacro (robot description, xacro)
@@ -12,5 +12,5 @@
     <xacro:property name="sensor_radius" value="0.0" /> <!-- [m] -->
     <!-- Included URDF Files (NEEDED FOR BASE SKIN UNIT) -->
-    <xacro:include filename="$(find gentact_descriptions)/robots/common/skin_unit_base.xacro" />
+    <xacro:include filename="$(find gentact_descriptions_hybrid)/robots/common/skin_unit_base.xacro" />
     <!-- Instantiate dermis once -->
     <xacro:dermis_base_macro

File: robots/h1-2/skin/shoulder_yaw_R_skin.xacro (robot description, xacro)
@@ -12,5 +12,5 @@
     <xacro:property name="sensor_radius" value="0.0" /> <!-- [m] -->
     <!-- Included URDF Files (NEEDED FOR BASE SKIN UNIT) -->
-    <xacro:include filename="$(find gentact_descriptions)/robots/common/skin_unit_base.xacro" />
+    <xacro:include filename="$(find gentact_descriptions_hybrid)/robots/common/skin_unit_base.xacro" />
     <!-- Instantiate dermis once -->
     <xacro:dermis_base_macro

File: robots/h1-2/skin/torso_skin.xacro (robot description, xacro)
@@ -12,5 +12,5 @@
     <xacro:property name="sensor_radius" value="0.0" /> <!-- [m] -->
     <!-- Included URDF Files (NEEDED FOR BASE SKIN UNIT) -->
-    <xacro:include filename="$(find gentact_descriptions)/robots/common/skin_unit_base.xacro" />
+    <xacro:include filename="$(find gentact_descriptions_hybrid)/robots/common/skin_unit_base.xacro" />
     <!-- Instantiate dermis once -->
     <xacro:dermis_base_macro
