Commit message: rename pkg in fr3_hybrid_skin.xacro and add humanoid xacro w nick skin

File: robots/fr3/fr3_hybrid_skin.xacro (robot description, xacro)
@@ -1,5 +1,5 @@
 <?xml version='1.0' encoding='utf-8'?>
 <robot xmlns:xacro="http://www.ros.org/wiki/xacro" name="fr3">
-  <xacro:include filename="$(find gentact_descriptions)/robots/common/franka_robot.xacro"/>
+  <xacro:include filename="$(find gentact_descriptions_hybrid)/robots/common/franka_robot.xacro"/>
   <!--
     DEPRECATION NOTICE
@@ -43,5 +43,5 @@
   <xacro:arg name="gazebo_effort" default="false" />
   <!-- Name of the description package -->
-  <xacro:arg name="description_pkg" default="gentact_descriptions" />
+  <xacro:arg name="description_pkg" default="gentact_descriptions_hybrid" />
   <!-- Define arguments for skin configurations -->
   <xacro:arg name="link1_skin" default=""/>
@@ -57,8 +57,8 @@
   <xacro:property name="modified_prefix" value="${prefix + '_' if prefix else ''}"/>
   <xacro:franka_robot arm_id="fr3"
-                      joint_limits="${xacro.load_yaml('$(find gentact_descriptions)/robots/fr3/joint_limits.yaml')}"
-                      inertials="${xacro.load_yaml('$(find gentact_descriptions)/robots/fr3/inertials.yaml')}"
-                      kinematics="${xacro.load_yaml('$(find gentact_descriptions)/robots/fr3/kinematics.yaml')}"
-                      dynamics="${xacro.load_yaml('$(find gentact_descriptions)/robots/fr3/dynamics.yaml')}"
+                      joint_limits="${xacro.load_yaml('$(find gentact_descriptions_hybrid)/robots/fr3/joint_limits.yaml')}"
+                      inertials="${xacro.load_yaml('$(find gentact_descriptions_hybrid)/robots/fr3/inertials.yaml')}"
+                      kinematics="${xacro.load_yaml('$(find gentact_descriptions_hybrid)/robots/fr3/kinematics.yaml')}"
+                      dynamics="${xacro.load_yaml('$(find gentact_descriptions_hybrid)/robots/fr3/dynamics.yaml')}"
                       gazebo="$(arg gazebo)"
                       hand="$(arg hand)"

File: robots/h1-2/h1_2_handless_tof.xacro (robot description, xacro)
@@ -1,4 +1,5 @@
 <?xml version="1.0"?>
 <robot xmlns:xacro="http://www.ros.org/wiki/xacro" name="h1_2">
+<!-- xacro for ToF Skins made by Nick J. -->
   <!-- Properties -->
   <xacro:property name="mesh_dir" value="meshes" />
@@ -376,8 +377,8 @@
     <limit lower="-2.35" upper="2.35" effort="200" velocity="23"/>
   </joint>
-  <xacro:include filename="skin/torso_skin.xacro" />
-  <xacro:torso_skin parent="torso_link" namespace="torso" />
-  <xacro:include filename="skin/head_skin.xacro" />
-  <xacro:head_skin parent="torso_link" namespace="head" />
+  <!-- <xacro:include filename="skin/torso_skin.xacro" /> -->
+  <!-- <xacro:torso_skin parent="torso_link" namespace="torso" /> -->
+  <!-- <xacro:include filename="skin/head_skin.xacro" /> -->
+  <!-- <xacro:head_skin parent="torso_link" namespace="head" /> -->
   <!-- L arm -->
   <link name="left_shoulder_pitch_link">
@@ -435,6 +436,6 @@
     <limit lower="-0.38" upper="3.4" effort="40" velocity="9"/>
   </joint>
-  <xacro:include filename="./skin/shoulder_roll_L_skin.xacro" />
-  <xacro:shoulder_roll_L_skin parent="left_shoulder_roll_link" namespace="left_shoulder_roll" />
+  <!-- <xacro:include filename="./skin/shoulder_roll_L_skin.xacro" /> -->
+  <!-- <xacro:shoulder_roll_L_skin parent="left_shoulder_roll_link" namespace="left_shoulder_roll" /> -->
   <link name="left_shoulder_yaw_link">
     <inertial>
@@ -464,6 +465,6 @@
     <limit lower="-2.66" upper="3.01" effort="18" velocity="20"/>
   </joint>
-  <xacro:include filename="./skin/shoulder_yaw_L_skin.xacro" />
-  <xacro:shoulder_yaw_L_skin parent="left_shoulder_yaw_link" namespace="left_shoulder_yaw" />
+  <!-- <xacro:include filename="./skin/shoulder_yaw_L_skin.xacro" /> -->
+  <!-- <xacro:shoulder_yaw_L_skin parent="left_shoulder_yaw_link" namespace="left_shoulder_yaw" /> -->
   <link name="left_elbow_link">
     <inertial>
@@ -493,6 +494,6 @@
     <limit lower="-0.95" upper="3.18" effort="18" velocity="20"/>
   </joint>
-  <xacro:include filename="./skin/elbow_L_skin.xacro" />
-  <xacro:elbow_L_skin parent="left_elbow_link" namespace="left_elbow" />
+  <!-- <xacro:include filename="./skin/elbow_L_skin.xacro" /> -->
+  <!-- <xacro:elbow_L_skin parent="left_elbow_link" namespace="left_elbow" /> -->
   <link name="left_wrist_roll_link">
     <inertial>
@@ -629,5 +630,6 @@
     <limit lower="-3.4" upper="0.38" effort="40" velocity="9"/>
   </joint>
-  <xacro:include filename="./skin/shoulder_roll_R_skin.xacro" />
+<!-- Shoulder Roll R Skin -->
+  <xacro:include filename="./skin/tof/shoulder_roll_R_skin.xacro" />
   <xacro:shoulder_roll_R_skin parent="right_shoulder_roll_link" namespace="right_shoulder_roll" />
   <link name="right_shoulder_yaw_link">
@@ -658,6 +660,6 @@
     <limit lower="-3.01" upper="2.66" effort="18" velocity="20"/>
   </joint>
-  <xacro:include filename="./skin/shoulder_yaw_R_skin.xacro" />
-  <xacro:shoulder_yaw_R_skin parent="right_shoulder_yaw_link" namespace="right_shoulder_yaw" />
+  <!-- <xacro:include filename="./skin/shoulder_yaw_R_skin.xacro" /> -->
+  <!-- <xacro:shoulder_yaw_R_skin parent="right_shoulder_yaw_link" namespace="right_shoulder_yaw" /> -->
   <link name="right_elbow_link">
     <inertial>
@@ -687,6 +689,6 @@
     <limit lower="-0.95" upper="3.18" effort="18" velocity="20"/>
   </joint>
-  <xacro:include filename="./skin/elbow_R_skin.xacro" />
-  <xacro:elbow_R_skin parent="right_elbow_link" namespace="right_elbow" />
+  <!-- <xacro:include filename="./skin/elbow_R_skin.xacro" /> -->
+  <!-- <xacro:elbow_R_skin parent="right_elbow_link" namespace="right_elbow" /> -->
   <link name="right_wrist_roll_link">
     <inertial>
@@ -805,3 +807,2 @@
   </joint>
 </robot>
-cock

File: robots/skin/hybrid/link2_hybrid.xacro (robot description, xacro)
@@ -25,29 +25,29 @@
     </xacro:dermis_base_macro>
     <!-- Instantiate sensors -->
-    <xacro:self_cap_sensor robot_namespace="${namespace}" parent="${namespace}_skin" sensor_number="0"
+    <xacro:self_cap_sensor robot_namespace="${namespace}" parent="${namespace}_skin" sensor_number="3"
       sensor_radius="${sensor_radius}" sensor_length="${sensor_length}" normal_x="0.723" normal_y="0.688" normal_z="-0.056">
       <origin xyz="0.052 0.111 -0.004" rpy="1.627 -0.000 2.332" />
     </xacro:self_cap_sensor>
-    <xacro:self_cap_sensor robot_namespace="${namespace}" parent="${namespace}_skin" sensor_number="1"
+    <xacro:self_cap_sensor robot_namespace="${namespace}" parent="${namespace}_skin" sensor_number="4"
       sensor_radius="${sensor_radius}" sensor_length="${sensor_length}" normal_x="0.458" normal_y="0.631" normal_z="0.627">
       <origin xyz="0.029 0.112 0.042" rpy="0.893 0.000 2.514" />
     </xacro:self_cap_sensor>
-    <xacro:self_cap_sensor robot_namespace="${namespace}" parent="${namespace}_skin" sensor_number="2"
+    <xacro:self_cap_sensor robot_namespace="${namespace}" parent="${namespace}_skin" sensor_number="0"
       sensor_radius="${sensor_radius}" sensor_length="${sensor_length}" normal_x="0.106" normal_y="0.989" normal_z="-0.108">
       <origin xyz="0.007 0.136 -0.007" rpy="-1.463 -3.142 -0.106" />
     </xacro:self_cap_sensor>
-    <xacro:self_cap_sensor robot_namespace="${namespace}" parent="${namespace}_skin" sensor_number="3"
+    <xacro:self_cap_sensor robot_namespace="${namespace}" parent="${namespace}_skin" sensor_number="5"
       sensor_radius="${sensor_radius}" sensor_length="${sensor_length}" normal_x="0.222" normal_y="0.969" normal_z="0.105">
       <origin xyz="0.009 0.064 0.131" rpy="1.466 0.000 2.917" />
     </xacro:self_cap_sensor>
-    <xacro:self_cap_sensor robot_namespace="${namespace}" parent="${namespace}_skin" sensor_number="4"
+    <xacro:self_cap_sensor robot_namespace="${namespace}" parent="${namespace}_skin" sensor_number="6"
       sensor_radius="${sensor_radius}" sensor_length="${sensor_length}" normal_x="-0.133" normal_y="0.605" normal_z="-0.785">
       <origin xyz="-0.009 0.112 -0.051" rpy="-0.668 -3.142 0.217" />
     </xacro:self_cap_sensor>
-    <xacro:self_cap_sensor robot_namespace="${namespace}" parent="${namespace}_skin" sensor_number="5"
+    <xacro:self_cap_sensor robot_namespace="${namespace}" parent="${namespace}_skin" sensor_number="1"
       sensor_radius="${sensor_radius}" sensor_length="${sensor_length}" normal_x="-0.341" normal_y="0.683" normal_z="0.646">
       <origin xyz="-0.024 0.113 0.045" rpy="0.869 -0.000 -2.678" />
     </xacro:self_cap_sensor>
-    <xacro:self_cap_sensor robot_namespace="${namespace}" parent="${namespace}_skin" sensor_number="6"
+    <xacro:self_cap_sensor robot_namespace="${namespace}" parent="${namespace}_skin" sensor_number="2"
       sensor_radius="${sensor_radius}" sensor_length="${sensor_length}" normal_x="-0.777" normal_y="0.627" normal_z="-0.060">
       <origin xyz="-0.050 0.113 -0.009" rpy="1.630 -0.000 -2.249" />

File: robots/skin/hybrid/link5_hybrid_back.xacro (robot description, xacro)
@@ -1,9 +1,9 @@
 <?xml version="1.0"?>
 <robot xmlns:xacro="http://ros.org/wiki/xacro">
-  <!-- Macro definition for link5 pt 2 skin -->
+  <!-- Macro definition for link5 pt 1 skin -->
   <xacro:macro name="link5_back_skin" params="parent namespace">
     <!-- Properties -->
     <xacro:property name="use_mesh_file" value="true" />
-    <xacro:property name="mesh_file" value="package://gentact_descriptions_hybrid/meshes/skin/hybrid/link5_part2_hybrid_dermis.stl" />
+    <xacro:property name="mesh_file" value="package://gentact_descriptions_hybrid/meshes/skin/hybrid/link5_part1_hybrid_dermis.stl" />
     <xacro:property name="mass" value="0.3" /> <!-- [kg] -->
     <xacro:property name="body_width" value="0.3" /> <!-- [m] -->

File: robots/skin/hybrid/link5_hybrid_front.xacro (robot description, xacro)
@@ -1,9 +1,9 @@
 <?xml version="1.0"?>
 <robot xmlns:xacro="http://ros.org/wiki/xacro">
-  <!-- Macro definition for link5 pt 1 skin -->
+  <!-- Macro definition for link5 pt 2 skin -->
   <xacro:macro name="link5_front_skin" params="parent namespace">
     <!-- Properties -->
     <xacro:property name="use_mesh_file" value="true" />
-    <xacro:property name="mesh_file" value="package://gentact_descriptions_hybrid/meshes/skin/hybrid/link5_part1_hybrid_dermis.stl" />
+    <xacro:property name="mesh_file" value="package://gentact_descriptions_hybrid/meshes/skin/hybrid/link5_part2_hybrid_dermis.stl" />
     <xacro:property name="mass" value="0.3" /> <!-- [kg] -->
     <xacro:property name="body_width" value="0.3" /> <!-- [m] -->
