Commit message: add correct sensor positions to xacro h1_2

File: robots/go-1/xacro/skin/thigh_skin.xacro (robot description, xacro)
@@ -30,8 +30,8 @@
         sensor_radius="${sensor_radius}"
         sensor_length="0.0"
-        normal_x="1.643"
-        normal_y="0.053"
-        normal_z="-0.634">
-        <origin xyz="-0.045 -0.011 -0.005" rpy="1.643 0.053 -0.634" />
+        normal_x="-0.0033466597087681293"
+        normal_y="-0.9991910457611084"
+        normal_z="-0.04007663577795029">
+        <origin xyz="-0.0054705264046788216 -0.01703549548983574 -0.02506975084543228" rpy="1.6108835935592651 3.0750507695742613e-10 -0.003349356586113572" />
     </xacro:self_cap_sensor>
     <xacro:self_cap_sensor
@@ -41,8 +41,8 @@
         sensor_radius="${sensor_radius}"
         sensor_length="0.0"
-        normal_x="1.078"
-        normal_y="-0.020"
-        normal_z="-0.037">
-        <origin xyz="-0.001 -0.013 0.042" rpy="1.078 -0.020 -0.037" />
+        normal_x="0.03249296545982361"
+        normal_y="-0.9906070828437805"
+        normal_z="0.1328226923942566">
+        <origin xyz="0.09776215255260468 -0.009773069061338902 -0.003952523693442345" rpy="1.4375799894332886 -2.939074983387968e-09 0.032789308577775955" />
     </xacro:self_cap_sensor>
     <xacro:self_cap_sensor
@@ -52,8 +52,8 @@
         sensor_radius="${sensor_radius}"
         sensor_length="0.0"
-        normal_x="0.944"
-        normal_y="-3.130"
-        normal_z="0.055">
-        <origin xyz="0.002 -0.012 -0.044" rpy="2.198 -0.022 0.031" />
+        normal_x="0.13000711798667908"
+        normal_y="-0.9857586622238159"
+        normal_z="0.10666757822036743">
+        <origin xyz="0.02981957234442234 -0.015662170946598053 0.0170421302318573" rpy="1.4639254808425903 -1.415918404745753e-08 0.13112856447696686" />
     </xacro:self_cap_sensor>
     <xacro:self_cap_sensor
@@ -63,8 +63,8 @@
         sensor_radius="${sensor_radius}"
         sensor_length="0.0"
-        normal_x="1.572"
-        normal_y="-0.000"
-        normal_z="0.017">
-        <origin xyz="0.002 -0.017 -0.003" rpy="1.572 -0.000 0.017" />
+        normal_x="0.12371029704809189"
+        normal_y="-0.8856444358825684"
+        normal_z="-0.4475819766521454">
+        <origin xyz="0.03183375298976898 -0.012470245361328125 -0.038558200001716614" rpy="2.034855842590332 1.6719945428178562e-09 0.1387859433889389" />
     </xacro:self_cap_sensor>
     <xacro:self_cap_sensor
@@ -74,8 +74,8 @@
         sensor_radius="${sensor_radius}"
         sensor_length="0.0"
-        normal_x="1.570"
-        normal_y="0.000"
-        normal_z="0.144">
-        <origin xyz="0.048 -0.014 -0.005" rpy="1.570 0.000 0.144" />
+        normal_x="0.06528738886117935"
+        normal_y="-0.5346206426620483"
+        normal_z="0.8425664901733398">
+        <origin xyz="0.09520145505666733 0.008756054565310478 0.02564341574907303" rpy="0.5687653422355652 -1.8162769066520923e-08 0.12151739746332169" />
     </xacro:self_cap_sensor>
     <xacro:self_cap_sensor
@@ -85,8 +85,8 @@
         sensor_radius="${sensor_radius}"
         sensor_length="0.0"
-        normal_x="1.542"
-        normal_y="0.000"
-        normal_z="0.017">
-        <origin xyz="0.095 -0.010 -0.008" rpy="1.542 0.000 0.017" />
+        normal_x="0.004111784510314465"
+        normal_y="-0.9999915361404419"
+        normal_z="2.02366391022224e-06">
+        <origin xyz="-0.006869952194392681 -0.017091382294893265 0.005429353564977646" rpy="1.5707944631576538 2.0792034760575007e-10 0.004111796617507935" />
     </xacro:self_cap_sensor>
     <xacro:self_cap_sensor
@@ -96,8 +96,8 @@
         sensor_radius="${sensor_radius}"
         sensor_length="0.0"
-        normal_x="0.179"
-        normal_y="0.036"
-        normal_z="0.007">
-        <origin xyz="0.089 0.021 0.031" rpy="0.179 0.036 0.007" />
+        normal_x="0.00975038856267929"
+        normal_y="0.10503476858139038"
+        normal_z="0.9944207668304443">
+        <origin xyz="0.08788560330867767 0.03748124837875366 0.03188776969909668" rpy="0.10568315535783768 -2.4437664336574016e-08 3.049027919769287" />
     </xacro:self_cap_sensor>
     <xacro:self_cap_sensor
@@ -107,8 +107,19 @@
         sensor_radius="${sensor_radius}"
         sensor_length="0.0"
-        normal_x="3.032"
-        normal_y="-0.022"
-        normal_z="0.002">
-        <origin xyz="0.089 0.026 -0.054" rpy="3.032 -0.022 0.002" />
+        normal_x="0.049779538065195084"
+        normal_y="-0.26070669293403625"
+        normal_z="-0.9641338586807251">
+        <origin xyz="0.08021856844425201 0.01752631552517414 -0.05247209593653679" rpy="2.8729567527770996 -1.6629815746682652e-08 0.188669815659523" />
+    </xacro:self_cap_sensor>
+    <xacro:self_cap_sensor
+        robot_namespace="${namespace}"
+        parent="${namespace}_skin"
+        sensor_number="8"
+        sensor_radius="${sensor_radius}"
+        sensor_length="0.0"
+        normal_x="0.15267664194107056"
+        normal_y="-0.8526670932769775"
+        normal_z="-0.4996485412120819">
+        <origin xyz="0.06785736232995987 -0.006429128348827362 -0.03632089123129845" rpy="2.093989372253418 -2.5215447507775934e-09 0.17718012630939484" />
     </xacro:self_cap_sensor>
     </xacro:macro>

File: robots/h1-2/skin/tof/elbow_R_skin.xacro (robot description, xacro)
@@ -30,8 +30,8 @@
         sensor_radius="${sensor_radius}"
         sensor_length="0.0"
-        normal_x="-0.0033466597087681293"
-        normal_y="-0.9991910457611084"
-        normal_z="-0.04007663577795029">
-        <origin xyz="-0.0054705264046788216 -0.01703549548983574 -0.02506975084543228" rpy="1.6108835935592651 3.0750507695742613e-10 -0.003349356586113572" />
+        normal_x="1.643"
+        normal_y="0.053"
+        normal_z="-0.634">
+        <origin xyz="-0.045 -0.011 -0.005" rpy="1.643 0.053 -0.634" />
     </xacro:self_cap_sensor>
     <xacro:self_cap_sensor
@@ -41,8 +41,8 @@
         sensor_radius="${sensor_radius}"
         sensor_length="0.0"
-        normal_x="0.03249296545982361"
-        normal_y="-0.9906070828437805"
-        normal_z="0.1328226923942566">
-        <origin xyz="0.09776215255260468 -0.009773069061338902 -0.003952523693442345" rpy="1.4375799894332886 -2.939074983387968e-09 0.032789308577775955" />
+        normal_x="1.078"
+        normal_y="-0.020"
+        normal_z="-0.037">
+        <origin xyz="-0.001 -0.013 0.042" rpy="1.078 -0.020 -0.037" />
     </xacro:self_cap_sensor>
     <xacro:self_cap_sensor
@@ -52,8 +52,8 @@
         sensor_radius="${sensor_radius}"
         sensor_length="0.0"
-        normal_x="0.13000711798667908"
-        normal_y="-0.9857586622238159"
-        normal_z="0.10666757822036743">
-        <origin xyz="0.02981957234442234 -0.015662170946598053 0.0170421302318573" rpy="1.4639254808425903 -1.415918404745753e-08 0.13112856447696686" />
+        normal_x="0.944"
+        normal_y="-3.130"
+        normal_z="0.055">
+        <origin xyz="0.002 -0.012 -0.044" rpy="2.198 -0.022 0.031" />
     </xacro:self_cap_sensor>
     <xacro:self_cap_sensor
@@ -63,8 +63,8 @@
         sensor_radius="${sensor_radius}"
         sensor_length="0.0"
-        normal_x="0.12371029704809189"
-        normal_y="-0.8856444358825684"
-        normal_z="-0.4475819766521454">
-        <origin xyz="0.03183375298976898 -0.012470245361328125 -0.038558200001716614" rpy="2.034855842590332 1.6719945428178562e-09 0.1387859433889389" />
+        normal_x="1.572"
+        normal_y="-0.000"
+        normal_z="0.017">
+        <origin xyz="0.002 -0.017 -0.003" rpy="1.572 -0.000 0.017" />
     </xacro:self_cap_sensor>
     <xacro:self_cap_sensor
@@ -74,8 +74,8 @@
         sensor_radius="${sensor_radius}"
         sensor_length="0.0"
-        normal_x="0.06528738886117935"
-        normal_y="-0.5346206426620483"
-        normal_z="0.8425664901733398">
-        <origin xyz="0.09520145505666733 0.008756054565310478 0.02564341574907303" rpy="0.5687653422355652 -1.8162769066520923e-08 0.12151739746332169" />
+        normal_x="1.570"
+        normal_y="0.000"
+        normal_z="0.144">
+        <origin xyz="0.048 -0.014 -0.005" rpy="1.570 0.000 0.144" />
     </xacro:self_cap_sensor>
     <xacro:self_cap_sensor
@@ -85,8 +85,8 @@
         sensor_radius="${sensor_radius}"
         sensor_length="0.0"
-        normal_x="0.004111784510314465"
-        normal_y="-0.9999915361404419"
-        normal_z="2.02366391022224e-06">
-        <origin xyz="-0.006869952194392681 -0.017091382294893265 0.005429353564977646" rpy="1.5707944631576538 2.0792034760575007e-10 0.004111796617507935" />
+        normal_x="1.542"
+        normal_y="0.000"
+        normal_z="0.017">
+        <origin xyz="0.095 -0.010 -0.008" rpy="1.542 0.000 0.017" />
     </xacro:self_cap_sensor>
     <xacro:self_cap_sensor
@@ -96,8 +96,8 @@
         sensor_radius="${sensor_radius}"
         sensor_length="0.0"
-        normal_x="0.00975038856267929"
-        normal_y="0.10503476858139038"
-        normal_z="0.9944207668304443">
-        <origin xyz="0.08788560330867767 0.03748124837875366 0.03188776969909668" rpy="0.10568315535783768 -2.4437664336574016e-08 3.049027919769287" />
+        normal_x="0.179"
+        normal_y="0.036"
+        normal_z="0.007">
+        <origin xyz="0.089 0.021 0.031" rpy="0.179 0.036 0.007" />
     </xacro:self_cap_sensor>
     <xacro:self_cap_sensor
@@ -107,19 +107,8 @@
         sensor_radius="${sensor_radius}"
         sensor_length="0.0"
-        normal_x="0.049779538065195084"
-        normal_y="-0.26070669293403625"
-        normal_z="-0.9641338586807251">
-        <origin xyz="0.08021856844425201 0.01752631552517414 -0.05247209593653679" rpy="2.8729567527770996 -1.6629815746682652e-08 0.188669815659523" />
-    </xacro:self_cap_sensor>
-    <xacro:self_cap_sensor
-        robot_namespace="${namespace}"
-        parent="${namespace}_skin"
-        sensor_number="8"
-        sensor_radius="${sensor_radius}"
-        sensor_length="0.0"
-        normal_x="0.15267664194107056"
-        normal_y="-0.8526670932769775"
-        normal_z="-0.4996485412120819">
-        <origin xyz="0.06785736232995987 -0.006429128348827362 -0.03632089123129845" rpy="2.093989372253418 -2.5215447507775934e-09 0.17718012630939484" />
+        normal_x="3.032"
+        normal_y="-0.022"
+        normal_z="0.002">
+        <origin xyz="0.089 0.026 -0.054" rpy="3.032 -0.022 0.002" />
     </xacro:self_cap_sensor>
     </xacro:macro>

File: robots/h1-2/skin/tof/shoulder_yaw_R_skin.xacro (robot description, xacro)
@@ -30,8 +30,8 @@
         sensor_radius="${sensor_radius}"
         sensor_length="0.0"
-        normal_x="0.9508576989173889"
-        normal_y="-0.12113388627767563"
-        normal_z="-0.28494971990585327">
-        <origin xyz="0.04118751734495163 -0.004814512562006712 -0.08737954497337341" rpy="1.8597503900527954 1.1286831025358879e-08 1.4440847635269165" />
+        normal_x="-1.586"
+        normal_y="-0.062"
+        normal_z="1.796">
+        <origin xyz="-0.052 -0.011 -0.040" rpy="1.586 0.067 -1.345" />
     </xacro:self_cap_sensor>
     <xacro:self_cap_sensor
@@ -41,8 +41,8 @@
         sensor_radius="${sensor_radius}"
         sensor_length="0.0"
-        normal_x="-0.6932508945465088"
-        normal_y="-0.7167385220527649"
-        normal_z="-0.07542620599269867">
-        <origin xyz="-0.035796575248241425 -0.03355425223708153 -0.04064032435417175" rpy="1.646294355392456 1.8119585831755103e-09 -0.7687416672706604" />
+        normal_x="1.641"
+        normal_y="1.629"
+        normal_z="-1.218">
+        <origin xyz="-0.051 -0.012 -0.092" rpy="1.567 -0.014 -1.288" />
     </xacro:self_cap_sensor>
     <xacro:self_cap_sensor
@@ -52,8 +52,8 @@
         sensor_radius="${sensor_radius}"
         sensor_length="0.0"
-        normal_x="0.04019082337617874"
-        normal_y="-0.9604589939117432"
-        normal_z="-0.2755054235458374">
-        <origin xyz="0.0068807341158390045 -0.038329385221004486 -0.07258914411067963" rpy="1.8499118089675903 -2.4386073160798105e-09 0.04182104021310806" />
+        normal_x="-0.259"
+        normal_y="-1.757"
+        normal_z="1.398">
+        <origin xyz="-0.028 -0.039 -0.069" rpy="1.751 0.082 -0.421" />
     </xacro:self_cap_sensor>
     <xacro:self_cap_sensor
@@ -63,8 +63,8 @@
         sensor_radius="${sensor_radius}"
         sensor_length="0.0"
-        normal_x="-0.9944165349006653"
-        normal_y="-0.10552489757537842"
-        normal_z="-0.0004047837865073234">
-        <origin xyz="-0.04953809827566147 -0.003564621554687619 -0.0796278566122055" rpy="1.571201205253601 3.790614400145387e-08 -1.4650746583938599" />
+        normal_x="1.390"
+        normal_y="-3.116"
+        normal_z="0.091">
+        <origin xyz="0.006 -0.049 -0.043" rpy="1.751 -0.015 0.084" />
     </xacro:self_cap_sensor>
     <xacro:self_cap_sensor
@@ -74,8 +74,8 @@
         sensor_radius="${sensor_radius}"
         sensor_length="0.0"
-        normal_x="-0.13521844148635864"
-        normal_y="0.9906842708587646"
-        normal_z="0.01614234782755375">
-        <origin xyz="-0.00878828577697277 0.04951019585132599 -0.0318453386425972" rpy="1.5546531677246094 -2.4349319005523284e-08 -3.0059409141540527" />
+        normal_x="1.410"
+        normal_y="-3.101"
+        normal_z="0.006">
+        <origin xyz="0.003 -0.033 -0.106" rpy="1.731 0.000 -0.001" />
     </xacro:self_cap_sensor>
     <xacro:self_cap_sensor
@@ -85,8 +85,19 @@
         sensor_radius="${sensor_radius}"
         sensor_length="0.0"
-        normal_x="-0.16762951016426086"
-        normal_y="-0.9856319427490234"
-        normal_z="-0.020739588886499405">
-        <origin xyz="-0.0280979685485363 -0.027626603841781616 -0.11977264285087585" rpy="1.5915374755859375 1.0039254760840777e-08 -0.16846124827861786" />
+        normal_x="1.814"
+        normal_y="0.018"
+        normal_z="0.641">
+        <origin xyz="0.032 -0.034 -0.072" rpy="1.818 -0.171 0.594" />
+    </xacro:self_cap_sensor>
+    <xacro:self_cap_sensor
+        robot_namespace="${namespace}"
+        parent="${namespace}_skin"
+        sensor_number="6"
+        sensor_radius="${sensor_radius}"
+        sensor_length="0.0"
+        normal_x="1.584"
+        normal_y="-0.029"
+        normal_z="1.136">
+        <origin xyz="0.049 -0.021 -0.038" rpy="1.584 -0.029 1.136" />
     </xacro:self_cap_sensor>
     </xacro:macro>
