Commit message: fix urdf (thighcap pose)

File: robots/go-1/xacro/skin/left_thighcap_skin.xacro (robot description, xacro)
@@ -5,5 +5,5 @@
     <!-- Properties -->
     <xacro:property name="use_mesh_file" value="true" />
-    <xacro:property name="mesh_file" value="${mesh_dir}skin/thighcap/left_thighcap_skin.stl" />
+    <xacro:property name="mesh_file" value="${mesh_dir}skin/thigh/left_thighcap_skin.stl" />
     <xacro:property name="mass" value="0.0" /> <!-- [kg] -->
     <xacro:property name="body_width" value="0.0" /> <!-- [m] -->
@@ -33,5 +33,5 @@
         normal_y="1.224162220954895"
         normal_z="1.6694881916046143">
-        <origin xyz="0.006742224097251892 0.014293902553617954 0.029223144054412842" rpy="-1.2252006530761719 -0.005685813259333372 0.0157905425876379" />
+        <origin xyz="0.0010693295625969768 -0.006162808742374182 0.046794019639492035" rpy="-1.2252006530761719 -0.005685813259333372 0.0157905425876379" />
     </xacro:self_cap_sensor>
     <xacro:self_cap_sensor
@@ -44,5 +44,5 @@
         normal_y="0.6460541486740112"
         normal_z="1.1572322845458984">
-        <origin xyz="-0.037725191563367844 -0.0013956413604319096 0.008954118005931377" rpy="-1.3508657217025757 -0.3039449453353882 0.9292620420455933" />
+        <origin xyz="-0.0425979383289814 -0.008709190413355827 0.021811174228787422" rpy="-1.3508657217025757 -0.3039449453353882 0.9292620420455933" />
     </xacro:self_cap_sensor>
     <xacro:self_cap_sensor
@@ -55,5 +55,5 @@
         normal_y="2.012662410736084"
         normal_z="1.626475214958191">
-        <origin xyz="0.0007210002513602376 0.013414165005087852 -0.016765158623456955" rpy="-2.012596607208252 0.012588809244334698 0.026608869433403015" />
+        <origin xyz="-0.004939308390021324 0.01649658940732479 0.0077791460789740086" rpy="-2.012596607208252 0.012588809244334698 0.026608869433403015" />
     </xacro:self_cap_sensor>
     </xacro:macro>

File: robots/go-1/xacro/skin/right_thighcap_skin.xacro (robot description, xacro)
@@ -5,5 +5,5 @@
     <!-- Properties -->
     <xacro:property name="use_mesh_file" value="true" />
-    <xacro:property name="mesh_file" value="${mesh_dir}skin/thighcap/right_thighcap_skin.stl" />
+    <xacro:property name="mesh_file" value="${mesh_dir}skin/thigh/right_thighcap_skin.stl" />
     <xacro:property name="mass" value="0.0" /> <!-- [kg] -->
     <xacro:property name="body_width" value="0.0" /> <!-- [m] -->
@@ -33,5 +33,5 @@
         normal_y="1.224162220954895"
         normal_z="1.6694881916046143">
-        <origin xyz="0.006742224097251892 -0.014293902553617954 0.029223144054412842" rpy="-1.2252006530761719 -0.005685813259333372 0.0157905425876379" />
+        <origin xyz="0.0010693295625969768 0.007912559434771538 0.046794019639492035" rpy="-1.2252006530761719 -0.005685813259333372 0.0157905425876379" />
     </xacro:self_cap_sensor>
     <xacro:self_cap_sensor
@@ -44,5 +44,5 @@
         normal_y="0.6460541486740112"
         normal_z="1.1572322845458984">
-        <origin xyz="-0.037725191563367844 0.0013956413604319096 0.008954118005931377" rpy="-1.3508657217025757 -0.3039449453353882 0.9292620420455933" />
+        <origin xyz="-0.0425979383289814 0.009698150679469109 0.021811174228787422" rpy="-1.3508657217025757 -0.3039449453353882 0.9292620420455933" />
     </xacro:self_cap_sensor>
     <xacro:self_cap_sensor
@@ -55,5 +55,5 @@
         normal_y="2.012662410736084"
         normal_z="1.626475214958191">
-        <origin xyz="0.0007210002513602376 -0.013414165005087852 -0.016765158623456955" rpy="-2.012596607208252 0.012588809244334698 0.026608869433403015" />
+        <origin xyz="-0.004939308390021324 -0.01481604017317295 0.0077791460789740086" rpy="-2.012596607208252 0.012588809244334698 0.026608869433403015" />
     </xacro:self_cap_sensor>
     </xacro:macro>

File: robots/go-1/xacro/skin/trunk_head_skin.xacro (robot description, xacro)
@@ -22,5 +22,5 @@
     use_mesh_file="${use_mesh_file}"
     mesh_file="${mesh_file}">
-    <origin xyz="0 0 0" rpy="0 0 0" />
+    <origin xyz="0.275155 0.001302 0.010202" rpy="0 0 1.570796" />
     </xacro:dermis_base_macro>
     <xacro:self_cap_sensor
@@ -30,8 +30,8 @@
         sensor_radius="${sensor_radius}"
         sensor_length="0.0"
-        normal_x="-1.5642733573913574"
-        normal_y="-0.0002883475972339511"
-        normal_z="0.0441758893430233">
-        <origin xyz="-0.020546915009617805 0.016203830018639565 -0.13735900819301605" rpy="-1.5642733573913574 -0.0002883475972339511 0.0441758893430233" />
+        normal_x="1.2075234651565552"
+        normal_y="-0.007908201776444912"
+        normal_z="-0.020799949765205383">
+        <origin xyz="0.00025236696819774806 -0.2968325912952423 0.04981664940714836" rpy="1.2075234651565552 -0.007908201776444912 -0.020799949765205383" />
     </xacro:self_cap_sensor>
     <xacro:self_cap_sensor
@@ -41,8 +41,8 @@
         sensor_radius="${sensor_radius}"
         sensor_length="0.0"
-        normal_x="-1.6060417890548706"
-        normal_y="-0.0003777451638597995"
-        normal_z="-0.010712702758610249">
-        <origin xyz="-0.00846764538437128 0.016201069578528404 -0.046428292989730835" rpy="-1.6060417890548706 -0.0003777451638597995 -0.010712702758610249" />
+        normal_x="1.1489475965499878"
+        normal_y="-0.39848679304122925"
+        normal_z="-0.7129077315330505">
+        <origin xyz="-0.03770412877202034 -0.2818562388420105 0.051483239978551865" rpy="1.1489475965499878 -0.39848679304122925 -0.7129077315330505" />
     </xacro:self_cap_sensor>
     <xacro:self_cap_sensor
@@ -52,8 +52,30 @@
         sensor_radius="${sensor_radius}"
         sensor_length="0.0"
-        normal_x="1.6190142631530762"
-        normal_y="-0.024614643305540085"
-        normal_z="-1.5761873722076416">
-        <origin xyz="-0.0421280711889267 0.000184581644134596 -0.10028665512800217" rpy="-2.077631950378418 1.4713668823242188 1.0618557929992676" />
+        normal_x="1.1440706253051758"
+        normal_y="0.4009367823600769"
+        normal_z="0.7093470692634583">
+        <origin xyz="0.03843432292342186 -0.28169137239456177 0.05167349427938461" rpy="1.1440706253051758 0.4009367823600769 0.7093470692634583" />
+    </xacro:self_cap_sensor>
+    <xacro:self_cap_sensor
+        robot_namespace="${namespace}"
+        parent="${namespace}_skin"
+        sensor_number="3"
+        sensor_radius="${sensor_radius}"
+        sensor_length="0.0"
+        normal_x="1.494691252708435"
+        normal_y="-0.024021487683057785"
+        normal_z="-0.30515751242637634">
+        <origin xyz="-0.06460931897163391 -0.27623823285102844 0.0038362115155905485" rpy="1.494691252708435 -0.024021487683057785 -0.30515751242637634" />
+    </xacro:self_cap_sensor>
+    <xacro:self_cap_sensor
+        robot_namespace="${namespace}"
+        parent="${namespace}_skin"
+        sensor_number="4"
+        sensor_radius="${sensor_radius}"
+        sensor_length="0.0"
+        normal_x="1.4878184795379639"
+        normal_y="0.02471890300512314"
+        normal_z="0.2888708710670471">
+        <origin xyz="0.06688925623893738 -0.2754700481891632 0.00686574075371027" rpy="1.4878184795379639 0.02471890300512314 0.2888708710670471" />
     </xacro:self_cap_sensor>
     </xacro:macro>
