Commit message: fix head sensor poses

File: robots/go-1/xacro/skin/trunk_head_skin.xacro (robot description, xacro)
@@ -22,5 +22,5 @@
     use_mesh_file="${use_mesh_file}"
     mesh_file="${mesh_file}">
-    <origin xyz="0.275155 0.001302 0.010202" rpy="0 0 1.570796" />
+    <origin xyz="0 0 0" rpy="0 0 0" />
     </xacro:dermis_base_macro>
     <xacro:self_cap_sensor
@@ -33,5 +33,5 @@
         normal_y="-0.007908201776444912"
         normal_z="-0.020799949765205383">
-        <origin xyz="0.00025236696819774806 -0.2968325912952423 0.04981664940714836" rpy="1.2075234651565552 -0.007908201776444912 -0.020799949765205383" />
+        <origin xyz="0.29396241903305054 -0.0024843034334480762 0.04981664940714836" rpy="1.2075234651565552 -0.007908201776444912 -0.020799949765205383" />
     </xacro:self_cap_sensor>
     <xacro:self_cap_sensor
@@ -44,5 +44,5 @@
         normal_y="-0.39848679304122925"
         normal_z="-0.7129077315330505">
-        <origin xyz="-0.03770412877202034 -0.2818562388420105 0.051483239978551865" rpy="1.1489475965499878 -0.39848679304122925 -0.7129077315330505" />
+        <origin xyz="0.2779468894004822 -0.03731217980384827 0.051483239978551865" rpy="1.1489475965499878 -0.39848679304122925 -0.7129077315330505" />
     </xacro:self_cap_sensor>
     <xacro:self_cap_sensor
@@ -55,5 +55,5 @@
         normal_y="0.4009367823600769"
         normal_z="0.7093470692634583">
-        <origin xyz="0.03843432292342186 -0.28169137239456177 0.05167349427938461" rpy="1.1440706253051758 0.4009367823600769 0.7093470692634583" />
+        <origin xyz="0.28208127617836 0.03453124314546585 0.05167349427938461" rpy="1.1440706253051758 0.4009367823600769 0.7093470692634583" />
     </xacro:self_cap_sensor>
     <xacro:self_cap_sensor
@@ -66,5 +66,5 @@
         normal_y="-0.024021487683057785"
         normal_z="-0.30515751242637634">
-        <origin xyz="-0.06460931897163391 -0.27623823285102844 0.0038362115155905485" rpy="1.494691252708435 -0.024021487683057785 -0.30515751242637634" />
+        <origin xyz="0.27248281240463257 -0.06655683368444443 0.0038362115155905485" rpy="1.494691252708435 -0.024021487683057785 -0.30515751242637634" />
     </xacro:self_cap_sensor>
     <xacro:self_cap_sensor
@@ -77,5 +77,5 @@
         normal_y="0.02471890300512314"
         normal_z="0.2888708710670471">
-        <origin xyz="0.06688925623893738 -0.2754700481891632 0.00686574075371027" rpy="1.4878184795379639 0.02471890300512314 0.2888708710670471" />
+        <origin xyz="0.27346357703208923 0.06316765397787094 0.00686574075371027" rpy="1.4878184795379639 0.02471890300512314 0.2888708710670471" />
     </xacro:self_cap_sensor>
     </xacro:macro>
