Commit message: add go-1 xacros

File: robots/go-1/xacro/depthCamera.xacro (robot description, xacro)
@@ -17,5 +17,5 @@
             <origin xyz="0 0 0" rpy="0 0 0"/>
             <geometry>
-                <mesh filename="package://go1_description/meshes/depthCamera.dae" scale="1 1 1"/>
+                <mesh filename="${mesh_dir}depthCamera.dae" scale="1 1 1"/>
             </geometry>
             </visual>

File: robots/go-1/xacro/leg.xacro (robot description, xacro)
@@ -1,5 +1,5 @@
 <?xml version="1.0"?>
 <robot xmlns:xacro="http://www.ros.org/wiki/xacro">
-    <xacro:include filename="$(find go1_description)/xacro/transmission.xacro"/>
+    <xacro:include filename="./transmission.xacro"/>
     <xacro:macro name="leg" params="name mirror mirror_dae front_hind front_hind_dae">
         <joint name="${name}_hip_joint" type="revolute">
@@ -58,5 +58,5 @@
                 </xacro:if>
                 <geometry>
-                    <mesh filename="package://go1_description/meshes/hip.dae" scale="1 1 1"/>
+                    <mesh filename="${mesh_dir}hip.dae" scale="1 1 1"/>
                 </geometry>
                 <!-- <material name="orange"/> -->
@@ -118,8 +118,8 @@
                 <geometry>
                     <xacro:if value="${mirror_dae == True}">
-                        <mesh filename="package://go1_description/meshes/thigh.dae" scale="1 1 1"/>
+                        <mesh filename="${mesh_dir}thigh.dae" scale="1 1 1"/>
                     </xacro:if>
                     <xacro:if value="${mirror_dae == False}">
-                        <mesh filename="package://go1_description/meshes/thigh_mirror.dae" scale="1 1 1"/>
+                        <mesh filename="${mesh_dir}thigh_mirror.dae" scale="1 1 1"/>
                     </xacro:if>
                 </geometry>
@@ -181,5 +181,5 @@
                 <origin rpy="0 0 0" xyz="0 0 0"/>
                 <geometry>
-                    <mesh filename="package://go1_description/meshes/calf.dae" scale="1 1 1"/>
+                    <mesh filename="${mesh_dir}calf.dae" scale="1 1 1"/>
                 </geometry>
                 <!-- <material name="orange"/> -->

File: robots/go-1/xacro/robot.xacro (robot description, xacro)
@@ -2,12 +2,13 @@
 <robot name="go1" xmlns:xacro="http://www.ros.org/wiki/xacro">
     <xacro:arg name="DEBUG" default="false"/>
-    <xacro:include filename="$(find go1_description)/xacro/const.xacro"/>
-    <xacro:include filename="$(find go1_description)/xacro/materials.xacro"/>
-    <xacro:include filename="$(find go1_description)/xacro/leg.xacro"/>
-    <!-- <xacro:include filename="$(find go1_description)/xacro/stairs.xacro"/> -->
-    <xacro:include filename="$(find go1_description)/xacro/gazebo.xacro"/>
-    <xacro:include filename="$(find go1_description)/xacro/depthCamera.xacro"/>
-    <xacro:include filename="$(find go1_description)/xacro/ultraSound.xacro"/>
-    <!-- <xacro:include filename="$(find go1_gazebo)/launch/stairs.urdf.xacro"/> -->
+    <xacro:property name="mesh_dir" value="package://gentact_ros_tools_hybrid/meshes/go-1/" />
+    <xacro:include filename="./const.xacro"/>
+    <xacro:include filename="./materials.xacro"/>
+    <xacro:include filename="./leg.xacro"/>
+    <!-- <xacro:include filename="./stairs.xacro"/> -->
+    <xacro:include filename="./gazebo.xacro"/>
+    <xacro:include filename="./depthCamera.xacro"/>
+    <xacro:include filename="./ultraSound.xacro"/>
+    <!-- <xacro:include filename="./launch/stairs.urdf.xacro"/> -->
     <!-- <xacro:stairs stairs="15" xpos="0" ypos="0" zpos="0" /> -->
     <!-- Rotor related joint and link is only for demonstrate location. -->
@@ -39,5 +40,5 @@
             <origin rpy="0 0 0" xyz="0 0 0"/>
             <geometry>
-                <mesh filename="package://go1_description/meshes/trunk.dae" scale="1 1 1"/>
+                <mesh filename="${mesh_dir}trunk.dae" scale="1 1 1"/>
             </geometry>
             <!-- <material name="orange"/> -->
@@ -58,4 +59,7 @@
         </inertial>
     </link>
+    <xacro:include filename="./skin/trunk_head_skin.xacro" />
+    <!-- namespace is trunk_head so that sensor names are trunk_head_skin -->
+    <xacro:trunk_head_skin parent="base" namespace="trunk_head" />
     <joint name="imu_joint" type="fixed">
         <parent link="trunk"/>
@@ -87,4 +91,16 @@
     <xacro:leg name="RR" mirror="-1" mirror_dae="False"  front_hind="-1" front_hind_dae="False" />
     <xacro:leg name="RL" mirror="1"  mirror_dae="True"   front_hind="-1" front_hind_dae="False" />
+    <xacro:include filename="./skin/left_calf_skin.xacro" />
+    <xacro:left_calf_skin parent="FL_calf" namespace="left_calf" />
+    <xacro:include filename="./skin/right_calf_skin.xacro" />
+    <xacro:right_calf_skin parent="FR_calf" namespace="right_calf" />
+    <xacro:include filename="./skin/left_thighcap_skin.xacro" />
+    <xacro:left_thighcap_skin parent="FL_thigh" namespace="left_thighcap" />
+    <xacro:include filename="./skin/right_thighcap_skin.xacro" />
+    <xacro:right_thighcap_skin parent="FR_thigh" namespace="right_thighcap" />
+    <xacro:include filename="./skin/left_thigh_skin.xacro" />
+    <xacro:left_thigh_skin parent="FL_thigh" namespace="left_thigh" />
+    <xacro:include filename="./skin/right_thigh_skin.xacro" />
+    <xacro:right_thigh_skin parent="FR_thigh" namespace="right_thigh" />
     <xacro:depthCamera camID="1" name="face">
         <origin rpy="${PI} 0 0" xyz="0.2785 0.0125 0.0167"/>

File: robots/go-1/xacro/ultraSound.xacro (robot description, xacro)
@@ -17,5 +17,5 @@
             <origin xyz="0 0 0" rpy="0 0 0"/>
             <geometry>
-                <mesh filename="package://go1_description/meshes/ultraSound.dae" scale="1 1 1"/>
+                <mesh filename="${mesh_dir}ultraSound.dae" scale="1 1 1"/>
             </geometry>
             <material name="black"/>

File: robots/h1-2/h1_2_handless_tof.xacro (robot description, xacro)
@@ -35,12 +35,12 @@
       <origin xyz="0 0 0" rpy="0 0 0"/>
       <geometry>
-        <mesh filename="${mesh_dir}/pelvis.STL"/>
-      </geometry>
-      <xacro:material_grey />
-    </visual>
-    <collision>
-      <origin xyz="0 0 0" rpy="0 0 0"/>
-      <geometry>
-        <mesh filename="${mesh_dir}/pelvis.STL"/>
+        <mesh filename="${mesh_dir}pelvis.STL"/>
+      </geometry>
+      <xacro:material_grey />
+    </visual>
+    <collision>
+      <origin xyz="0 0 0" rpy="0 0 0"/>
+      <geometry>
+        <mesh filename="${mesh_dir}pelvis.STL"/>
       </geometry>
     </collision>
@@ -56,5 +56,5 @@
       <origin xyz="0 0 0" rpy="0 0 0"/>
       <geometry>
-        <mesh filename="${mesh_dir}/left_hip_yaw_link.STL"/>
+        <mesh filename="${mesh_dir}left_hip_yaw_link.STL"/>
       </geometry>
       <xacro:material_grey />
@@ -77,12 +77,12 @@
       <origin xyz="0 0 0" rpy="0 0 0"/>
       <geometry>
-        <mesh filename="${mesh_dir}/left_hip_pitch_link.STL"/>
-      </geometry>
-      <xacro:material_grey />
-    </visual>
-    <collision>
-      <origin xyz="0 0 0" rpy="0 0 0"/>
-      <geometry>
-        <mesh filename="${mesh_dir}/left_hip_pitch_link.STL"/>
+        <mesh filename="${mesh_dir}left_hip_pitch_link.STL"/>
+      </geometry>
+      <xacro:material_grey />
+    </visual>
+    <collision>
+      <origin xyz="0 0 0" rpy="0 0 0"/>
+      <geometry>
+        <mesh filename="${mesh_dir}left_hip_pitch_link.STL"/>
       </geometry>
     </collision>
@@ -104,12 +104,12 @@
       <origin xyz="0 0 0" rpy="0 0 0"/>
       <geometry>
-        <mesh filename="${mesh_dir}/left_hip_roll_link.STL"/>
-      </geometry>
-      <xacro:material_grey />
-    </visual>
-    <collision>
-      <origin xyz="0 0 0" rpy="0 0 0"/>
-      <geometry>
-        <mesh filename="${mesh_dir}/left_hip_roll_link.STL"/>
+        <mesh filename="${mesh_dir}left_hip_roll_link.STL"/>
+      </geometry>
+      <xacro:material_grey />
+    </visual>
+    <collision>
+      <origin xyz="0 0 0" rpy="0 0 0"/>
+      <geometry>
+        <mesh filename="${mesh_dir}left_hip_roll_link.STL"/>
       </geometry>
     </collision>
@@ -131,5 +131,5 @@
       <origin xyz="0 0 0" rpy="0 0 0"/>
       <geometry>
-        <mesh filename="${mesh_dir}/left_knee_link.STL"/>
+        <mesh filename="${mesh_dir}left_knee_link.STL"/>
       </geometry>
       <xacro:material_grey />
@@ -160,5 +160,5 @@
       <origin xyz="0 0 0" rpy="0 0 0"/>
       <geometry>
-        <mesh filename="${mesh_dir}/left_ankle_pitch_link.STL"/>
+        <mesh filename="${mesh_dir}left_ankle_pitch_link.STL"/>
       </geometry>
       <xacro:material_grey />
@@ -181,12 +181,12 @@
       <origin xyz="0 0 0" rpy="0 0 0"/>
       <geometry>
-        <mesh filename="${mesh_dir}/left_ankle_roll_link.STL"/>
-      </geometry>
-      <xacro:material_grey />
-    </visual>
-    <collision>
-      <origin xyz="0 0 0" rpy="0 0 0"/>
-      <geometry>
-        <mesh filename="${mesh_dir}/left_ankle_roll_link.STL"/>
+        <mesh filename="${mesh_dir}left_ankle_roll_link.STL"/>
+      </geometry>
+      <xacro:material_grey />
+    </visual>
+    <collision>
+      <origin xyz="0 0 0" rpy="0 0 0"/>
+      <geometry>
+        <mesh filename="${mesh_dir}left_ankle_roll_link.STL"/>
       </geometry>
     </collision>
@@ -211,5 +211,5 @@
       <origin xyz="0 0 0" rpy="0 0 0"/>
       <geometry>
-        <mesh filename="${mesh_dir}/right_hip_yaw_link.STL"/>
+        <mesh filename="${mesh_dir}right_hip_yaw_link.STL"/>
       </geometry>
       <xacro:material_grey />
@@ -232,12 +232,12 @@
       <origin xyz="0 0 0" rpy="0 0 0"/>
       <geometry>
-        <mesh filename="${mesh_dir}/right_hip_pitch_link.STL"/>
-      </geometry>
-      <xacro:material_grey />
-    </visual>
-    <collision>
-      <origin xyz="0 0 0" rpy="0 0 0"/>
-      <geometry>
-        <mesh filename="${mesh_dir}/right_hip_pitch_link.STL"/>
+        <mesh filename="${mesh_dir}right_hip_pitch_link.STL"/>
+      </geometry>
+      <xacro:material_grey />
+    </visual>
+    <collision>
+      <origin xyz="0 0 0" rpy="0 0 0"/>
+      <geometry>
+        <mesh filename="${mesh_dir}right_hip_pitch_link.STL"/>
       </geometry>
     </collision>
@@ -259,12 +259,12 @@
       <origin xyz="0 0 0" rpy="0 0 0"/>
       <geometry>
-        <mesh filename="${mesh_dir}/right_hip_roll_link.STL"/>
-      </geometry>
-      <xacro:material_grey />
-    </visual>
-    <collision>
-      <origin xyz="0 0 0" rpy="0 0 0"/>
-      <geometry>
-        <mesh filename="${mesh_dir}/right_hip_roll_link.STL"/>
+        <mesh filename="${mesh_dir}right_hip_roll_link.STL"/>
+      </geometry>
+      <xacro:material_grey />
+    </visual>
+    <collision>
+      <origin xyz="0 0 0" rpy="0 0 0"/>
+      <geometry>
+        <mesh filename="${mesh_dir}right_hip_roll_link.STL"/>
       </geometry>
     </collision>
@@ -288,5 +288,5 @@
       <origin xyz="0 0 0" rpy="0 0 0"/>
       <geometry>
-        <mesh filename="${mesh_dir}/right_knee_link.STL"/>
+        <mesh filename="${mesh_dir}right_knee_link.STL"/>
       </geometry>
       <xacro:material_grey />
@@ -317,5 +317,5 @@
       <origin xyz="0 0 0" rpy="0 0 0"/>
       <geometry>
-        <mesh filename="${mesh_dir}/right_ankle_pitch_link.STL"/>
+        <mesh filename="${mesh_dir}right_ankle_pitch_link.STL"/>
       </geometry>
       <xacro:material_grey />
@@ -338,12 +338,12 @@
       <origin xyz="0 0 0" rpy="0 0 0"/>
       <geometry>
-        <mesh filename="${mesh_dir}/right_ankle_roll_link.STL"/>
-      </geometry>
-      <xacro:material_grey />
-    </visual>
-    <collision>
-      <origin xyz="0 0 0" rpy="0 0 0"/>
-      <geometry>
-        <mesh filename="${mesh_dir}/right_ankle_roll_link.STL"/>
+        <mesh filename="${mesh_dir}right_ankle_roll_link.STL"/>
+      </geometry>
+      <xacro:material_grey />
+    </visual>
+    <collision>
+      <origin xyz="0 0 0" rpy="0 0 0"/>
+      <geometry>
+        <mesh filename="${mesh_dir}right_ankle_roll_link.STL"/>
       </geometry>
     </collision>
@@ -366,12 +366,12 @@
       <origin xyz="0 0 0" rpy="0 0 0"/>
       <geometry>
-        <mesh filename="${mesh_dir}/torso_link.STL"/>
-      </geometry>
-      <xacro:material_grey />
-    </visual>
-    <collision>
-      <origin xyz="0 0 0" rpy="0 0 0"/>
-      <geometry>
-        <mesh filename="${mesh_dir}/torso_link.STL"/>
+        <mesh filename="${mesh_dir}torso_link.STL"/>
+      </geometry>
+      <xacro:material_grey />
+    </visual>
+    <collision>
+      <origin xyz="0 0 0" rpy="0 0 0"/>
+      <geometry>
+        <mesh filename="${mesh_dir}torso_link.STL"/>
       </geometry>
     </collision>
@@ -400,12 +400,12 @@
       <origin xyz="0 0 0" rpy="0 0 0"/>
       <geometry>
-        <mesh filename="${mesh_dir}/left_shoulder_pitch_link.STL"/>
-      </geometry>
-      <xacro:material_grey />
-    </visual>
-    <collision>
-      <origin xyz="0 0 0" rpy="0 0 0"/>
-      <geometry>
-        <mesh filename="${mesh_dir}/left_shoulder_pitch_link.STL"/>
+        <mesh filename="${mesh_dir}left_shoulder_pitch_link.STL"/>
+      </geometry>
+      <xacro:material_grey />
+    </visual>
+    <collision>
+      <origin xyz="0 0 0" rpy="0 0 0"/>
+      <geometry>
+        <mesh filename="${mesh_dir}left_shoulder_pitch_link.STL"/>
       </geometry>
     </collision>
@@ -427,12 +427,12 @@
       <origin xyz="0 0 0" rpy="0 0 0"/>
       <geometry>
-        <mesh filename="${mesh_dir}/left_shoulder_roll_link.STL"/>
-      </geometry>
-      <xacro:material_grey />
-    </visual>
-    <collision>
-      <origin xyz="0 0 0" rpy="0 0 0"/>
-      <geometry>
-        <mesh filename="${mesh_dir}/left_shoulder_roll_link.STL"/>
+        <mesh filename="${mesh_dir}left_shoulder_roll_link.STL"/>
+      </geometry>
+      <xacro:material_grey />
+    </visual>
+    <collision>
+      <origin xyz="0 0 0" rpy="0 0 0"/>
+      <geometry>
+        <mesh filename="${mesh_dir}left_shoulder_roll_link.STL"/>
       </geometry>
     </collision>
@@ -456,12 +456,12 @@
       <origin xyz="0 0 0" rpy="0 0 0"/>
       <geometry>
-        <mesh filename="${mesh_dir}/left_shoulder_yaw_link.STL"/>
-      </geometry>
-      <xacro:material_grey />
-    </visual>
-    <collision>
-      <origin xyz="0 0 0" rpy="0 0 0"/>
-      <geometry>
-        <mesh filename="${mesh_dir}/left_shoulder_yaw_link.STL"/>
+        <mesh filename="${mesh_dir}left_shoulder_yaw_link.STL"/>
+      </geometry>
+      <xacro:material_grey />
+    </visual>
+    <collision>
+      <origin xyz="0 0 0" rpy="0 0 0"/>
+      <geometry>
+        <mesh filename="${mesh_dir}left_shoulder_yaw_link.STL"/>
       </geometry>
     </collision>
@@ -485,12 +485,12 @@
       <origin xyz="0 0 0" rpy="0 0 0"/>
       <geometry>
-        <mesh filename="${mesh_dir}/left_elbow_link.STL"/>
-      </geometry>
-      <xacro:material_grey />
-    </visual>
-    <collision>
-      <origin xyz="0 0 0" rpy="0 0 0"/>
-      <geometry>
-        <mesh filename="${mesh_dir}/left_elbow_link.STL"/>
+        <mesh filename="${mesh_dir}left_elbow_link.STL"/>
+      </geometry>
+      <xacro:material_grey />
+    </visual>
+    <collision>
+      <origin xyz="0 0 0" rpy="0 0 0"/>
+      <geometry>
+        <mesh filename="${mesh_dir}left_elbow_link.STL"/>
       </geometry>
     </collision>
@@ -514,11 +514,11 @@
       <origin xyz="0 0 0" rpy="0 0 0"/>
       <geometry>
-        <mesh filename="${mesh_dir}/left_wrist_roll_link.STL"/>
-      </geometry>
-      <xacro:material_grey />
-    </visual>
-    <collision>
-      <geometry>
-        <mesh filename="${mesh_dir}/left_wrist_roll_link.STL"/>
+        <mesh filename="${mesh_dir}left_wrist_roll_link.STL"/>
+      </geometry>
+      <xacro:material_grey />
+    </visual>
+    <collision>
+      <geometry>
+        <mesh filename="${mesh_dir}left_wrist_roll_link.STL"/>
       </geometry>
     </collision>
@@ -540,11 +540,11 @@
       <origin xyz="0 0 0" rpy="0 0 0"/>
       <geometry>
-        <mesh filename="${mesh_dir}/left_wrist_pitch_link.STL"/>
-      </geometry>
-      <xacro:material_grey />
-    </visual>
-    <collision>
-      <geometry>
-        <mesh filename="${mesh_dir}/left_wrist_pitch_link.STL"/>
+        <mesh filename="${mesh_dir}left_wrist_pitch_link.STL"/>
+      </geometry>
+      <xacro:material_grey />
+    </visual>
+    <collision>
+      <geometry>
+        <mesh filename="${mesh_dir}left_wrist_pitch_link.STL"/>
       </geometry>
     </collision>
@@ -566,5 +566,5 @@
       <origin xyz="0 0 0" rpy="0 0 0"/>
       <geometry>
-        <mesh filename="${mesh_dir}/wrist_yaw_link.STL"/>
+        <mesh filename="${mesh_dir}wrist_yaw_link.STL"/>
       </geometry>
       <xacro:material_grey />
@@ -573,5 +573,5 @@
       <origin xyz="0 0 0" rpy="0 0 0"/>
       <geometry>
-        <mesh filename="${mesh_dir}/wrist_yaw_link.STL"/>
+        <mesh filename="${mesh_dir}wrist_yaw_link.STL"/>
       </geometry>
     </collision> -->
@@ -594,12 +594,12 @@
       <origin xyz="0 0 0" rpy="0 0 0"/>
       <geometry>
-        <mesh filename="${mesh_dir}/right_shoulder_pitch_link.STL"/>
-      </geometry>
-      <xacro:material_grey />
-    </visual>
-    <collision>
-      <origin xyz="0 0 0" rpy="0 0 0"/>
-      <geometry>
-        <mesh filename="${mesh_dir}/right_shoulder_pitch_link.STL"/>
+        <mesh filename="${mesh_dir}right_shoulder_pitch_link.STL"/>
+      </geometry>
+      <xacro:material_grey />
+    </visual>
+    <collision>
+      <origin xyz="0 0 0" rpy="0 0 0"/>
+      <geometry>
+        <mesh filename="${mesh_dir}right_shoulder_pitch_link.STL"/>
       </geometry>
     </collision>
@@ -621,12 +621,12 @@
       <origin xyz="0 0 0" rpy="0 0 0"/>
       <geometry>
-        <mesh filename="${mesh_dir}/right_shoulder_roll_link.STL"/>
-      </geometry>
-      <xacro:material_grey />
-    </visual>
-    <collision>
-      <origin xyz="0 0 0" rpy="0 0 0"/>
-      <geometry>
-        <mesh filename="${mesh_dir}/right_shoulder_roll_link.STL"/>
+        <mesh filename="${mesh_dir}right_shoulder_roll_link.STL"/>
+      </geometry>
+      <xacro:material_grey />
+    </visual>
+    <collision>
+      <origin xyz="0 0 0" rpy="0 0 0"/>
+      <geometry>
+        <mesh filename="${mesh_dir}right_shoulder_roll_link.STL"/>
       </geometry>
     </collision>
@@ -650,12 +650,12 @@
       <origin xyz="0 0 0" rpy="0 0 0"/>
       <geometry>
-        <mesh filename="${mesh_dir}/right_shoulder_yaw_link.STL"/>
-      </geometry>
-      <xacro:material_grey />
-    </visual>
-    <collision>
-      <origin xyz="0 0 0" rpy="0 0 0"/>
-      <geometry>
-        <mesh filename="${mesh_dir}/right_shoulder_yaw_link.STL"/>
+        <mesh filename="${mesh_dir}right_shoulder_yaw_link.STL"/>
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